File: 01_Hardware/RPiAutonomousCar.brd (EAGLE design)
At the start: 67.3 x 58.4 mm, 0 parts

Commit message: routing...
Parts:
- added JP1: (no value), pinhead:1X08
- added PCB1: RASPBERRY_PI_B+/PI2_DIM, RPiAutonomousCar:RASPBERRY_PI_BPLUS_DIM
- added U$1: TB6612FNG, RPiAutonomousCar:SSOP24
- added U1: TXB0108PWR, RPiAutonomousCar:SOP65P640X120-20N
Connections:
- new net +3V3: PCB1.1, U1.10, U1.2
- new net +5V: PCB1.2
- new net 3V3: PCB1.17
- new net 5V0: PCB1.4
- new net GND: PCB1.12, PCB1.14, PCB1.20, PCB1.25, PCB1.30, PCB1.34, PCB1.39, PCB1.6, PCB1.9, PCB1.PE_BL, PCB1.PE_TL, PCB1.PE_TR, U1.11
- new net N$1: JP1.1, U1.20
- new net N$14: PCB1.15
- new net N$2: JP1.2, U1.18
- new net N$3: JP1.3, U1.17
- new net N$4: JP1.4, U1.16
- new net N$5: JP1.5, U1.15
- new net N$6: JP1.6, U1.14
- new net N$7: JP1.7, U1.13
- new net N$8: JP1.8, U1.12
- new net SPI_CLK: PCB1.23
- new net SPI_MISO: PCB1.21
- new net SPI_MOSI: PCB1.19
- new net UART_RX: PCB1.10
- new net UART_TX: PCB1.8
- new net VCCB: U1.19
Routing:
- added copper zone on layer 1, net GND
- added copper zone on layer 16, net GND
Other:
- board text removed: "Chrg"
- board text removed: "Fault"
- board text removed: "N. Seidle"
- board text removed: "UserLED"
Changed lines of the file:
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@@
 <layer number="15" name="Route15" color="4" fill="6" visible="no" active="no"/>
 <layer number="16" name="Bottom" color="1" fill="1" visible="yes" active="yes"/>
-<layer number="17" name="Pads" color="2" fill="1" visible="no" active="yes"/>
-<layer number="18" name="Vias" color="2" fill="1" visible="no" active="yes"/>
-<layer number="19" name="Unrouted" color="6" fill="1" visible="no" active="yes"/>
+<layer number="17" name="Pads" color="2" fill="1" visible="yes" active="yes"/>
+<layer number="18" name="Vias" color="2" fill="1" visible="yes" active="yes"/>
+<layer number="19" name="Unrouted" color="6" fill="1" visible="yes" active="yes"/>
 <layer number="20" name="Dimension" color="15" fill="1" visible="yes" active="yes"/>
-<layer number="21" name="tPlace" color="16" fill="1" visible="no" active="yes"/>
-<layer number="22" name="bPlace" color="14" fill="1" visible="no" active="yes"/>
-<layer number="23" name="tOrigins" color="15" fill="1" visible="no" active="yes"/>
-<layer number="24" name="bOrigins" color="15" fill="1" visible="no" active="yes"/>
-<layer number="25" name="tNames" color="7" fill="1" visible="no" active="yes"/>
-<layer number="26" name="bNames" color="7" fill="1" visible="no" active="yes"/>
-<layer number="27" name="tValues" color="7" fill="1" visible="no" active="yes"/>
-<layer number="28" name="bValues" color="7" fill="1" visible="no" active="yes"/>
+<layer number="21" name="tPlace" color="16" fill="1" visible="yes" active="yes"/>
+<layer number="22" name="bPlace" color="14" fill="1" visible="yes" active="yes"/>
+<layer number="23" name="tOrigins" color="15" fill="1" visible="yes" active="yes"/>
+<layer number="24" name="bOrigins" color="15" fill="1" visible="yes" active="yes"/>
+<layer number="25" name="tNames" color="7" fill="1" visible="yes" active="yes"/>
+<layer number="26" name="bNames" color="7" fill="1" visible="yes" active="yes"/>
+<layer number="27" name="tValues" color="7" fill="1" visible="yes" active="yes"/>
+<layer number="28" name="bValues" color="7" fill="1" visible="yes" active="yes"/>
 <layer number="29" name="tStop" color="7" fill="3" visible="no" active="yes"/>
 <layer number="30" name="bStop" color="7" fill="6" visible="no" active="yes"/>
@@
 <layer number="43" name="vRestrict" color="2" fill="10" visible="no" active="yes"/>
 <layer number="44" name="Drills" color="7" fill="1" visible="no" active="yes"/>
-<layer number="45" name="Holes" color="7" fill="1" visible="no" active="yes"/>
+<layer number="45" name="Holes" color="7" fill="1" visible="yes" active="yes"/>
 <layer number="46" name="Milling" color="3" fill="1" visible="no" active="yes"/>
 <layer number="47" name="Measures" color="7" fill="1" visible="no" active="yes"/>
@@
 <board>
 <plain>
-<text x="22.86" y="-24.13" size="1.778" layer="27" font="vector" ratio="15">N. Seidle</text>
-<text x="63.119" y="41.021" size="0.8128" layer="21" font="vector" ratio="15">Fault</text>
 <wire x1="67.564" y1="4.191" x2="63.754" y2="0.381" width="0" layer="20" curve="-90"/>
 <wire x1="4.064" y1="0.381" x2="0.254" y2="4.191" width="0" layer="20" curve="-90"/>
@@
 <wire x1="67.564" y1="4.191" x2="67.564" y2="54.991" width="0" layer="20"/>
 <wire x1="4.064" y1="58.801" x2="63.754" y2="58.801" width="0" layer="20"/>
-<text x="62.738" y="46.609" size="0.8128" layer="21" font="vector" ratio="15">Chrg</text>
-<text x="1.905" y="11.049" size="0.508" layer="21" font="vector" ratio="15">UserLED</text>
 </plain>
 <attributes>
@@
 </autorouter>
 <elements>
+<element name="PCB1" library="RPiAutonomousCar" package="RASPBERRY_PI_BPLUS_DIM" value="RASPBERRY_PI_B+/PI2_DIM" x="0.254" y="0.508"/>
+<element name="U1" library="RPiAutonomousCar" package="SOP65P640X120-20N" value="TXB0108PWR" x="12.446" y="37.846">
+<attribute name="MPN" value="TXB0108PWR" x="12.446" y="37.846" size="1.778" layer="27" display="off"/>
+<attribute name="OC_FARNELL" value="1494945" x="12.446" y="37.846" size="1.778" layer="27" display="off"/>
+<attribute name="PACKAGE" value="TSSOP-20" x="12.446" y="37.846" size="1.778" layer="27" display="off"/>
+<attribute name="OC_NEWARK" value="27M1151" x="12.446" y="37.846" size="1.778" layer="27" display="off"/>
+<attribute name="SUPPLIER" value="Texas Instruments" x="12.446" y="37.846" size="1.778" layer="27" display="off"/>
+</element>
+<element name="JP1" library="pinhead" package="1X08" value="" x="27.432" y="36.576" rot="R270"/>
+<element name="U$1" library="RPiAutonomousCar" package="SSOP24" value="TB6612FNG" x="23.876" y="17.526" rot="R270"/>
 </elements>
 <signals>
+<signal name="3V3">
+<contactref element="PCB1" pad="17"/>
+</signal>
+<signal name="GND">
+<contactref element="PCB1" pad="6"/>
+<contactref element="PCB1" pad="14"/>
+<contactref element="PCB1" pad="20"/>
+<contactref element="PCB1" pad="34"/>
+<contactref element="PCB1" pad="39"/>
+<contactref element="PCB1" pad="PE_TR"/>
+<contactref element="PCB1" pad="PE_TL"/>
+<contactref element="PCB1" pad="PE_BL"/>
+<contactref element="PCB1" pad="9"/>
+<contactref element="PCB1" pad="25"/>
+<contactref element="PCB1" pad="30"/>
+<contactref element="PCB1" pad="12"/>
+<polygon width="0.4064" layer="16">
+<vertex x="0.508" y="58.928"/>
+<vertex x="67.564" y="58.928"/>
+<vertex x="67.564" y="0.508"/>
+<vertex x="0.508" y="0.508"/>
+</polygon>
+<polygon width="0.4064" layer="1">
+<vertex x="0.762" y="58.928"/>
+<vertex x="67.564" y="58.928"/>
+<vertex x="67.564" y="0.762"/>
+<vertex x="0.508" y="0.762"/>
+<vertex x="0.508" y="58.928"/>
+</polygon>
+<contactref element="U1" pad="11"/>
+</signal>
+<signal name="5V0">
+<contactref element="PCB1" pad="4"/>
+</signal>
+<signal name="VCCB">
+<contactref element="U1" pad="19"/>
+</signal>
+<signal name="+5V">
+<contactref element="PCB1" pad="2"/>
+</signal>
+<signal name="+3V3">
+<contactref element="PCB1" pad="1"/>
+<contactref element="U1" pad="2"/>
+<contactref element="U1" pad="10"/>
+<wire x1="9.525" y1="40.132" x2="9.894" y2="53.008" width="0" layer="19" extent="1-1"/>
+<wire x1="9.525" y1="34.925" x2="9.525" y2="40.132" width="0" layer="19" extent="1-1"/>
+</signal>
+<signal name="N$1">
+<contactref element="U1" pad="20"/>
+<contactref element="JP1" pad="1"/>
+<wire x1="15.367" y1="40.767" x2="27.432" y2="45.466" width="0" layer="19" extent="1-1"/>
+</signal>
+<signal name="N$2">
+<contactref element="U1" pad="18"/>
+<contactref element="JP1" pad="2"/>
+<wire x1="15.367" y1="39.4716" x2="27.432" y2="42.926" width="0" layer="19" extent="1-1"/>
+</signal>
+<signal name="N$3">
+<contactref element="U1" pad="17"/>
+<contactref element="JP1" pad="3"/>
+<wire x1="15.367" y1="38.8112" x2="27.432" y2="40.386" width="0" layer="19" extent="1-1"/>
+</signal>
+<signal name="N$4">
+<contactref element="U1" pad="16"/>
+<contactref element="JP1" pad="4"/>
+<wire x1="15.367" y1="38.1762" x2="27.432" y2="37.846" width="0" layer="19" extent="1-1"/>
+</signal>
+<signal name="N$5">
+<contactref element="U1" pad="15"/>
+<contactref element="JP1" pad="5"/>
+<wire x1="15.367" y1="37.5158" x2="27.432" y2="35.306" width="0" layer="19" extent="1-1"/>
+</signal>
+<signal name="N$6">
+<contactref element="U1" pad="14"/>
+<contactref element="JP1" pad="6"/>
+<wire x1="15.367" y1="36.8808" x2="27.432" y2="32.766" width="0" layer="19" extent="1-1"/>
+</signal>
+<signal name="N$7">
+<contactref element="U1" pad="13"/>
+<contactref element="JP1" pad="7"/>
+<wire x1="15.367" y1="36.2204" x2="27.432" y2="30.226" width="0" layer="19" extent="1-1"/>
+</signal>
+<signal name="N$8">
+<contactref element="U1" pad="12"/>
+<contactref element="JP1" pad="8"/>
+<wire x1="27.432" y1="27.686" x2="15.367" y2="35.56" width="0" layer="19" extent="1-1"/>
+</signal>
+<signal name="UART_TX">
+<contactref element="PCB1" pad="8"/>
+</signal>
+<signal name="UART_RX">
+<contactref element="PCB1" pad="10"/>
+</signal>
+<signal name="SPI_CLK">
+<contactref element="PCB1" pad="23"/>
+</signal>
+<signal name="SPI_MISO">
+<contactref element="PCB1" pad="21"/>
+</signal>
+<signal name="SPI_MOSI">
+<contactref element="PCB1" pad="19"/>
+</signal>
+<signal name="N$14">
+<contactref element="PCB1" pad="15"/>
+</signal>
 </signals>
 <errors>

Commit message: routing
Parts:
- added BATTERY, MOTOR1, MOTOR2: (no value), pinhead:1X02
- added C1, C10, C2, C3, C4, C6: 100n, rcl:C0603
- added C11, C7, C8, C9: 10n, rcl:C0603
- added C5: (no value), rcl:153CLV-0405
- added IC1: 7805TV, linear:TO220V
- added JP2: (no value), pinhead:2X20
- added JP3: (no value), pinhead:1X04
- added R11, R12, R3, R4, R5, R6, R8, R9: 1K, rcl:R0603
- added SERVO: (no value), pinhead:1X03
- added U2, U3: SN74LVC1G04DCKR, RPiAutonomousCar:SOT65P210X110-5N
- added U4: MCP3004-I/ST, RPiAutonomousCar:SOP65P640X120-14N
- moved U$1 33.0 mm to (50.0, 37.6), turned to 0 degrees
- moved JP1 15.8 mm to (13.7, 28.7), turned to 180 degrees
- moved U1 1.08 mm to (11.7, 37.1), turned to 270 degrees
Connections:
- removed net 3V3: PCB1.17
- removed net SPI_CLK: PCB1.23
- removed net SPI_MISO: PCB1.21
- removed net SPI_MOSI: PCB1.19
- removed net UART_RX: PCB1.10
- removed net UART_TX: PCB1.8
- removed net VCCB: U1.19
- new net +UB: BATTERY.2, C4.1, C5.+, IC1.1, U$1.13, U$1.14, U$1.24
- new net AN_CH0: JP3.1, R5.2
- new net AN_CH1: JP3.2, R3.2
- new net AN_CH2: JP3.3, R8.2
- new net AN_CH3: JP3.4, R11.2
- new net M1_DIR_INV: U$1.22, U2.4
- new net M1_OUT1: MOTOR1.1, U$1.1, U$1.2
- new net M1_OUT2: MOTOR1.2, U$1.5, U$1.6
- new net M2_DIR_INV: U$1.16, U3.4
- new net M2_OUT1: MOTOR2.1, U$1.11, U$1.12
- new net M2_OUT2: MOTOR2.2, U$1.7, U$1.8
- new net N$10: C2.2, U3.5
- new net N$11: C11.1, R5.1, R6.2, U4.1
- new net N$13: C7.1, R3.1, R4.2, U4.2
- new net N$15: C9.1, R11.1, R12.2, U4.4
- new net N$9: C1.2, U2.5
- new net RPI10: JP2.10, PCB1.10
- new net RPI11: JP2.11, PCB1.11
- new net RPI12: JP2.12, PCB1.12
- new net RPI13: JP2.13, PCB1.13
- new net RPI14: U1.8
- new net RPI15: JP2.15, PCB1.15, U1.9
- new net RPI16: JP2.16, PCB1.16
- new net RPI17: JP2.17
- new net RPI18: JP2.18, PCB1.18
- new net RPI19: JP2.19, PCB1.19, U1.1, U4.9
- new net RPI21: JP2.21, PCB1.21, U1.3, U4.10
- new net RPI22: JP2.22, PCB1.22
- new net RPI23: JP2.23, PCB1.23, U1.4, U4.11
- new net RPI24: JP2.24, PCB1.24, U1.5, U4.8
- new net RPI26: JP2.26, PCB1.26
- new net RPI27: JP2.27, PCB1.27
- new net RPI28: JP2.28, PCB1.28
- new net RPI29: JP2.29, PCB1.29, U$1.23
- new net RPI3: JP2.3, PCB1.3, U1.6
- new net RPI31: JP2.31, PCB1.31, U$1.21, U2.2
- new net RPI32: JP2.32, PCB1.32
- new net RPI33: JP2.33, PCB1.33, U$1.19
- new net RPI35: JP2.35, PCB1.35, U$1.17, U3.2
- new net RPI36: JP2.36, PCB1.36
- new net RPI37: JP2.37, PCB1.37, U$1.15
- new net RPI38: JP2.38, PCB1.38
- new net RPI40: JP2.40, PCB1.40
- new net RPI5: JP2.5, PCB1.5, U1.7
- new net RPI7: JP2.7, PCB1.7
- new net RPI8: JP2.8, PCB1.8
- new net SERVOPWM: SERVO.1
- net +3V3: now also C1.1, C2.1, C3.1, C6.1, JP2.1, PCB1.17, SERVO.2, U$1.20, U4.13, U4.14
- net +5V: now also C10.1, IC1.3, JP2.2, JP2.4, U1.19
- net GND: now also BATTERY.1, C10.2, C11.2, C3.2, C4.2, C5.-, C6.2, C7.2, C8.2, C9.2, IC1.2, JP2.14, JP2.20, JP2.25, JP2.30, JP2.34, JP2.39, JP2.6, JP2.9, R12.1, R4.1, R6.1, R9.1, SERVO.3, U$1.10, U$1.18, U$1.3, U$1.4, U$1.9, U2.3, U3.3, U4.12, U4.7; no longer PCB1.12
- net N$14: now also C8.1, R8.1, R9.2, U4.3; no longer PCB1.15

Commit message: routing
Parts:
- added C12, C13: 100n, rcl:C0603
- added I2C_JP2, I2C_JP3: (no value), pinhead:1X02
- added LED1: (no value), led:SML0603
- added R1: 1K, rcl:R0603
- added SJ1: (no value), jumper:SJ_2
- added SPI_JP2: (no value), pinhead:1X03
- R11: value 1K -> 10K
- R12: value 1K -> 22K
- moved C10 159.7 mm to (47.5, 33.8), turned to 180 degrees
- moved R8 136.3 mm to (28.4, 36.1), turned to 180 degrees
- moved R9 135.3 mm to (31.2, 35.3), turned to 90 degrees
- moved R12 128.3 mm to (31.2, 30.5), turned to 90 degrees
- moved C8 125.6 mm to (32.8, 35.6), turned to 270 degrees
- moved R4 125.2 mm to (30.7, 39.4), turned to 90 degrees
- moved R11 124.3 mm to (28.4, 32.0), turned to 180 degrees
- moved R3 121.1 mm to (28.4, 40.4), turned to 180 degrees
- moved C9 119.4 mm to (33.0, 30.5), turned to 270 degrees
- moved C7 117.8 mm to (32.3, 39.4), turned to 270 degrees
- moved C11 116.5 mm to (32.8, 42.7), turned to 270 degrees
- moved R6 112.6 mm to (31.2, 42.7), turned to 90 degrees
- moved R5 109.2 mm to (28.7, 43.4), turned to 180 degrees
- moved C6 93.2 mm to (63.8, 39.9)
- moved U2 55.0 mm to (60.7, 35.8), turned to 180 degrees
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Connections:
- new net N$12: LED1.C, R1.1
- new net N$16: LED1.A
- net +3V3: now also C12.1
- net +5V: now also C13.1
- net +UB: now also SJ1.3
- net AN_CH3: now also SJ1.1, SJ1.2
- net GND: now also C12.2, C13.2, R1.2; no longer PCB1.PE_BL, PCB1.PE_TL, PCB1.PE_TR
- net RPI19: now also SPI_JP2.3
- net RPI21: now also SPI_JP2.2
- net RPI23: now also SPI_JP2.1
- net RPI3: now also I2C_JP2.2, I2C_JP3.2
- net RPI5: now also I2C_JP2.1, I2C_JP3.1
Routing:
- net RPI12: track 0.00 -> 7.57 mm
- net RPI15: track 0.00 -> 7.52 mm
- net RPI5: track 0.00 -> 7.52 mm
- net RPI16: track 0.00 -> 7.51 mm
- net RPI38: track 0.00 -> 7.40 mm
- net RPI11: track 0.00 -> 7.37 mm
- net RPI7: track 0.00 -> 7.37 mm
- net RPI40: track 0.00 -> 7.28 mm
- net RPI28: track 0.00 -> 7.28 mm
- net RPI26: track 0.00 -> 7.28 mm
- net RPI3: track 0.00 -> 7.21 mm
- net RPI13: track 0.00 -> 7.21 mm
- net RPI21: track 0.00 -> 7.21 mm
- net RPI37: track 0.00 -> 7.13 mm
- net RPI24: track 0.00 -> 7.13 mm
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
Commit message: routing ...
Parts:
- removed BATTERY, I2C_JP2, I2C_JP3, MOTOR1, MOTOR2: (no value), pinhead:1X02
- removed C10: 100n, rcl:C0603
- removed IC1: 7805TV, linear:TO220V
- removed SERVO, SPI_JP2: (no value), pinhead:1X03
- added JP10, JP11, JP12: (no value), jumper:JP1
- added JP13, JP4, JP5, JP9: (no value), jumper:JP2
- added JP6, JP7, JP8: (no value), jumper:JP4
- JP1: device pinhead:1X08 -> jumper:JP1
- PCB1: device RPiAutonomousCar:RASPBERRY_PI_BPLUS_DIM -> RPiAutonomousCar:RASPBERRY_PI_BPLUS_HEADER_ONLY
- moved PCB1 37.1 mm to (31.8, 20.1)
- moved JP1 33.3 mm to (15.7, 8.89), turned to 180 degrees
- moved U1 25.7 mm to (10.2, 14.5)
- moved JP2 24.9 mm to (33.8, 23.4)
- moved JP3 24.7 mm to (22.9, 13.7)
- moved C7 24.6 mm to (33.0, 14.7)
- moved R4 24.6 mm to (31.5, 14.7)
- moved R3 24.6 mm to (29.0, 15.7)
- moved C13 24.4 mm to (9.14, 8.38), turned to 270 degrees
- moved C8 24.4 mm to (33.0, 11.2)
- moved C11 24.4 mm to (33.0, 18.3)
- moved R5 24.4 mm to (29.0, 19.1)
- moved R6 24.4 mm to (31.5, 18.3)
- moved R1 24.2 mm to (61.5, 23.6), turned to 0 degrees
- moved SJ1 24.0 mm to (33.8, 6.35)
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Connections:
- removed net RPI14: U1.8
- removed net RPI17: JP2.17
- removed net SERVOPWM: SERVO.1
- net +3V3: now also JP2.17, JP6.4, JP9.2; no longer SERVO.2
- net +5V: now also JP5.2; no longer C10.1, IC1.3
- net +UB: now also JP4.2; no longer BATTERY.2, IC1.1
- net GND: now also JP4.1, JP4.3, JP5.1, JP5.3, JP6.1, JP9.3; no longer BATTERY.1, C10.2, IC1.2, SERVO.3
- net M1_OUT1: now also JP10.1; no longer MOTOR1.1
- net M1_OUT2: now also JP10.2; no longer MOTOR1.2
- net M2_OUT1: now also JP11.1; no longer MOTOR2.1
- net M2_OUT2: now also JP11.2; no longer MOTOR2.2
- net N$1: now also JP8.4; no longer JP1.8
- net N$16: now also JP9.1; no longer LED1.A
- net N$2: now also JP8.3; no longer JP1.7
- net N$3: now also JP8.2; no longer JP1.6
- net N$4: now also JP8.1; no longer JP1.5
- net N$5: now also JP7.4; no longer JP1.4
- net N$6: now also JP7.3; no longer JP1.3
- net N$7: now also JP7.2; no longer JP1.2
- net N$8: now also JP7.1; no longer JP1.1
- net RPI10: now also U1.9
- net RPI15: no longer U1.9
- net RPI19: now also JP13.3; no longer SPI_JP2.3
- net RPI21: now also JP13.2; no longer SPI_JP2.2
- net RPI23: now also JP13.1; no longer SPI_JP2.1
- net RPI3: now also JP1.2, JP12.2; no longer I2C_JP2.2, I2C_JP3.2
- net RPI40: now also LED1.A
- net RPI5: now also JP1.1, JP12.1; no longer I2C_JP2.1, I2C_JP3.1
- net RPI8: now also U1.8
Routing:
- net +3V3: track 0.00 -> 43.3 mm
- net +5V: track 0.00 -> 29.1 mm
- net N$1: track 0.00 -> 11.0 mm
- net N$8: track 0.00 -> 9.19 mm
- net N$2: track 0.00 -> 8.76 mm
- net N$7: track 0.00 -> 7.78 mm
- net RPI40: track 7.28 -> 0.00 mm
- net N$3: track 0.00 -> 6.58 mm
- net N$6: track 0.00 -> 5.52 mm
- net N$4: track 0.00 -> 5.04 mm
- net N$5: track 0.00 -> 4.73 mm
- net RPI12: track 7.57 -> 7.07 mm
Other:
- board size 67.3 x 58.4 mm -> 67.3 x 34 mm

Commit message: routing ...
Parts:
- removed JP3: (no value), pinhead:1X04
- JP13: device jumper:JP2 -> jumper:JP4
- moved JP10 20.9 mm to (44.7, 17.0)
- moved JP11 20.7 mm to (44.7, 10.9)
- moved JP13 10.4 mm to (21.8, 6.10)
- moved JP9 8.89 mm to (17.5, 7.11), turned to 270 degrees
- moved JP1 7.19 mm to (10.4, 4.06), turned to 0 degrees
- moved JP12 7.19 mm to (13.5, 4.06)
- moved SJ1 6.71 mm to (28.4, 2.29)
- moved C9 6.51 mm to (31.8, 6.10), turned to 270 degrees
- moved R12 6.51 mm to (30.2, 6.10), turned to 90 degrees
- moved C12 6.12 mm to (9.91, 19.3), turned to 180 degrees
- moved C11 4.68 mm to (28.4, 17.3)
- moved R5 4.68 mm to (24.4, 18.0)
- moved R6 4.68 mm to (26.9, 17.3)
- moved R8 3.95 mm to (26.2, 9.40)
- moved U4 3.89 mm to (35.6, 14.7)
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Connections:
- removed net N$16: JP9.1
- removed net N$3: JP8.2, U1.14
- new net N$18: JP1.1, JP12.2, JP8.1, U1.15
- net AN_CH0: now also JP13.1; no longer JP3.1
- net AN_CH1: now also JP13.2; no longer JP3.2
- net AN_CH2: now also JP13.3; no longer JP3.3
- net AN_CH3: now also JP13.4; no longer JP3.4
- net N$4: now also JP1.2, JP12.1, JP8.2, U1.14; no longer JP8.1, U1.15
- net RPI19: no longer JP13.3
- net RPI21: no longer JP13.2
- net RPI23: no longer JP13.1
- net RPI26: now also JP6.3
- net RPI27: now also JP6.2
- net RPI3: no longer JP1.2, JP12.2
- net RPI5: no longer JP1.1, JP12.1
- net RPI7: now also JP9.1
Routing:
- net N$18: track 0.00 -> 25.2 mm
- net RPI26: track 7.07 -> 25.8 mm
- net RPI27: track 7.07 -> 25.4 mm
- net N$4: track 5.04 -> 22.9 mm
- net RPI7: track 7.07 -> 19.6 mm
- net +3V3: track 43.3 -> 33.7 mm
- net N$3: track 6.58 -> 0.00 mm
- net N$8: track 9.19 -> 11.7 mm
- net N$7: track 7.78 -> 7.19 mm
- net +5V: track 29.1 -> 29.6 mm, vias 0 -> 1

Commit message: rounting/Pinout minor changes
Parts:
- removed C1, C2: 100n, rcl:C0603
- removed U2, U3: SN74LVC1G04DCKR, RPiAutonomousCar:SOT65P210X110-5N
- moved C6 27.6 mm to (36.8, 15.5), turned to 90 degrees
- moved JP10 24.0 mm to (64.8, 3.81), turned to 0 degrees
- moved JP11 20.2 mm to (64.8, 8.89), turned to 180 degrees
- moved C5 14.7 mm to (43.2, 15.0), turned to 0 degrees
- moved C4 13.5 mm to (53.6, 6.86)
- moved C3 12.4 mm to (49.0, 11.4)
- moved U$1 5.68 mm to (56.4, 12.4), turned to 90 degrees
- moved U4 5.06 mm to (34.0, 9.91)
- moved R11 4.82 mm to (32.3, 5.33), turned to 270 degrees
- moved C9 4.20 mm to (35.6, 4.32)
- moved R12 4.20 mm to (34.0, 4.32)
- moved R5 4.17 mm to (26.9, 14.7), turned to 270 degrees
- moved R3 4.13 mm to (24.9, 10.4), turned to 270 degrees
- moved C8 4.10 mm to (28.4, 6.10)
- moved R9 4.10 mm to (26.9, 6.10)
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Connections:
- removed net M1_DIR_INV: U$1.22, U2.4
- removed net M2_DIR_INV: U$1.16, U3.4
- removed net N$10: C2.2, U3.5
- removed net N$9: C1.2, U2.5
- net +3V3: no longer C1.1, C2.1
- net GND: no longer U2.3, U3.3
- net RPI12: now also JP6.2
- net RPI13: now also JP6.3
- net RPI22: now also U4.8
- net RPI24: no longer U4.8
- net RPI26: no longer JP6.3
- net RPI27: no longer JP6.2
- net RPI31: no longer U2.2
- net RPI32: now also U$1.22
- net RPI35: no longer U3.2
- net RPI36: now also U$1.16
Routing:
- net +5V: track 29.6 -> 86.6 mm
- net RPI12: track 7.07 -> 38.3 mm
- net RPI13: track 7.37 -> 31.2 mm
- net +UB: track 0.00 -> 19.8 mm
- net RPI26: track 25.8 -> 7.07 mm
- net RPI27: track 25.4 -> 7.07 mm
- net RPI40: track 0.00 -> 13.1 mm
- net RPI8: track 7.07 -> 19.7 mm, vias 0 -> 1
- net RPI3: track 7.07 -> 19.5 mm, vias 0 -> 1
- net RPI7: track 19.6 -> 7.43 mm
- net RPI10: track 7.07 -> 19.0 mm
- net RPI5: track 7.22 -> 19.0 mm, vias 0 -> 1
- net AN_CH3: track 0.00 -> 10.3 mm
- net N$15: track 0.00 -> 9.90 mm
- net N$14: track 0.00 -> 8.60 mm
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
Commit message: routing almost done
Parts:
- moved C6 8.99 mm to (42.9, 8.89), turned to 270 degrees
- moved C3 3.89 mm to (45.2, 10.7), turned to 270 degrees
- moved C11 2.90 mm to (32.8, 14.0), turned to 0 degrees
- moved R5 1.08 mm to (27.7, 14.0)
- moved R6 1.08 mm to (29.2, 14.0)
- moved C5 1.02 mm to (43.2, 16.0)
Routing:
- net +3V3: track 42.0 -> 99.7 mm
- net RPI21: track 7.07 -> 43.4 mm
- net RPI24: track 7.07 -> 40.1 mm
- net RPI23: track 7.37 -> 36.9 mm
- net RPI19: track 7.22 -> 34.9 mm, vias 0 -> 1
- net +UB: track 19.8 -> 46.0 mm, vias 0 -> 2
- net RPI35: track 7.22 -> 25.1 mm, vias 0 -> 1
- net RPI36: track 7.07 -> 24.8 mm
- net RPI7: track 7.43 -> 21.0 mm
- net RPI33: track 7.22 -> 18.7 mm, vias 0 -> 1
- net M1_OUT1: track 0.00 -> 10.3 mm
- net M1_OUT2: track 0.00 -> 9.80 mm
- net RPI37: track 7.37 -> 17.1 mm
- net M2_OUT1: track 0.00 -> 9.27 mm
- net M2_OUT2: track 0.00 -> 8.83 mm

Commit message: routing done
Parts:
- moved C11 2.03 mm to (30.7, 14.0), turned to 270 degrees
- moved C6 1.93 mm to (43.7, 10.7)
- moved C4 1.27 mm to (52.6, 6.10)
- moved JP6 0.76 mm to (40.9, 6.10)
Routing:
- net RPI22: track 7.07 -> 27.1 mm, vias 0 -> 2
- net RPI32: track 7.07 -> 27.0 mm, vias 0 -> 1
- net RPI29: track 7.37 -> 26.0 mm, vias 0 -> 1
- net RPI31: track 7.07 -> 22.1 mm, vias 0 -> 1
- net RPI21: track 43.4 -> 54.7 mm, vias 0 -> 2
- net RPI19: track 34.9 -> 45.6 mm
- net RPI23: track 36.9 -> 46.6 mm, vias 0 -> 2
- net +3V3: track 99.7 -> 97.8 mm
- net RPI13: track 31.2 -> 32.4 mm
- net N$11: track 6.98 -> 8.03 mm
- net N$15: track 9.90 -> 9.09 mm
- net RPI12: track 38.3 -> 39.0 mm
