File: 01_Hardware/RPiAutonomousCar.sch (EAGLE design)
At the start: 0 parts

Commit message: routing...
Parts:
- added JP1: (no value), pinhead:PINHD-1X8
- added PCB1: RASPBERRY_PI_B+/PI2_DIM, RPiAutonomousCar:RASPBERRY_PI_B+/PI2_DIM
- added U$1: TB6612FNG, RPiAutonomousCar:TB6612FNG
- added U1: TXB0108PWR, RPiAutonomousCar:TXB0108PWR
Connections:
- new net +3V3: PCB1.3V3@1, U1.OE, U1.VCCA
- new net +5V: PCB1.5V0@1
- new net GND: PCB1.BL, PCB1.GND@1, PCB1.GND@2, PCB1.GND@3, PCB1.GND@5, PCB1.GND@6, PCB1.GND@7, PCB1.GND@8, PCB1.GPIO18, PCB1.TL, PCB1.TR, U1.GND
- new net N$1: JP1.1, U1.B1
- new net N$14: PCB1.GPIO22/GEN3
- new net N$2: JP1.2, U1.B2
- new net N$3: JP1.3, U1.B3
- new net N$4: JP1.4, U1.B4
- new net N$5: JP1.5, U1.B5
- new net N$6: JP1.6, U1.B6
- new net N$7: JP1.7, U1.B7
- new net N$8: JP1.8, U1.B8
- new net SPI_CLK: PCB1.GPIO11/SCLK
- new net SPI_MISO: PCB1.GPIO09/MISO
- new net SPI_MOSI: PCB1.GPIO10/MOSI
- new net UART_RX: PCB1.RXD0/GPIO15
- new net UART_TX: PCB1.TXD0/GPIO14
Changed lines of the file:
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@@
 <parts>
 <part name="FRAME1" library="frames" deviceset="DINA4_L" device=""/>
+<part name="PCB1" library="RPiAutonomousCar" deviceset="RASPBERRY_PI_B+/PI2" device="_DIM"/>
+<part name="GND1" library="supply1" deviceset="GND" device=""/>
+<part name="U1" library="RPiAutonomousCar" deviceset="TXB0108PWR" device=""/>
+<part name="GND2" library="supply1" deviceset="GND" device=""/>
+<part name="SUPPLY1" library="supply2" deviceset="+5V" device=""/>
+<part name="+3V1" library="supply1" deviceset="+3V3" device=""/>
+<part name="SUPPLY2" library="supply2" deviceset="+5V" device=""/>
+<part name="+3V2" library="supply1" deviceset="+3V3" device=""/>
+<part name="JP1" library="pinhead" deviceset="PINHD-1X8" device=""/>
+<part name="U$1" library="RPiAutonomousCar" deviceset="TB6612FNG" device=""/>
 </parts>
 <sheets>
@@
 <instance part="FRAME1" gate="G$1" x="0" y="0"/>
 <instance part="FRAME1" gate="G$2" x="162.56" y="0"/>
+<instance part="PCB1" gate="G$1" x="193.04" y="127"/>
+<instance part="GND1" gate="1" x="190.5" y="78.74"/>
+<instance part="U1" gate="A" x="38.1" y="109.22"/>
+<instance part="GND2" gate="1" x="17.78" y="78.74"/>
+<instance part="SUPPLY1" gate="+5V" x="218.44" y="160.02"/>
+<instance part="+3V1" gate="G$1" x="165.1" y="162.56"/>
+<instance part="SUPPLY2" gate="+5V" x="15.24" y="137.16"/>
+<instance part="+3V2" gate="G$1" x="20.32" y="132.08"/>
+<instance part="JP1" gate="A" x="71.12" y="111.76"/>
+<instance part="U$1" gate="G$1" x="109.22" y="144.78"/>
 </instances>
 <busses>
 </busses>
 <nets>
+<net name="GND" class="0">
+<segment>
+<pinref part="PCB1" gate="G$1" pin="TR"/>
+<pinref part="GND1" gate="1" pin="GND"/>
+<wire x1="190.5" y1="81.28" x2="190.5" y2="83.82" width="0.1524" layer="91"/>
+<pinref part="PCB1" gate="G$1" pin="TL"/>
+<wire x1="190.5" y1="83.82" x2="190.5" y2="86.36" width="0.1524" layer="91"/>
+<wire x1="185.42" y1="86.36" x2="185.42" y2="83.82" width="0.1524" layer="91"/>
+<wire x1="185.42" y1="83.82" x2="190.5" y2="83.82" width="0.1524" layer="91"/>
+<pinref part="PCB1" gate="G$1" pin="BL"/>
+<wire x1="190.5" y1="83.82" x2="195.58" y2="83.82" width="0.1524" layer="91"/>
+<wire x1="195.58" y1="83.82" x2="195.58" y2="86.36" width="0.1524" layer="91"/>
+<junction x="190.5" y="83.82"/>
+<wire x1="185.42" y1="83.82" x2="157.48" y2="83.82" width="0.1524" layer="91"/>
+<wire x1="157.48" y1="83.82" x2="157.48" y2="101.6" width="0.1524" layer="91"/>
+<pinref part="PCB1" gate="G$1" pin="GND@3"/>
+<wire x1="157.48" y1="101.6" x2="165.1" y2="101.6" width="0.1524" layer="91"/>
+<pinref part="PCB1" gate="G$1" pin="GND@1"/>
+<wire x1="165.1" y1="139.7" x2="157.48" y2="139.7" width="0.1524" layer="91"/>
+<wire x1="157.48" y1="139.7" x2="157.48" y2="119.38" width="0.1524" layer="91"/>
+<pinref part="PCB1" gate="G$1" pin="GND@2"/>
+<wire x1="157.48" y1="119.38" x2="165.1" y2="119.38" width="0.1524" layer="91"/>
+<wire x1="157.48" y1="119.38" x2="157.48" y2="101.6" width="0.1524" layer="91"/>
+<junction x="157.48" y="101.6"/>
+<junction x="157.48" y="119.38"/>
+<junction x="185.42" y="83.82"/>
+<pinref part="PCB1" gate="G$1" pin="GND@6"/>
+<wire x1="218.44" y1="114.3" x2="226.06" y2="114.3" width="0.1524" layer="91"/>
+<wire x1="195.58" y1="83.82" x2="226.06" y2="83.82" width="0.1524" layer="91"/>
+<wire x1="226.06" y1="83.82" x2="226.06" y2="109.22" width="0.1524" layer="91"/>
+<wire x1="226.06" y1="109.22" x2="226.06" y2="114.3" width="0.1524" layer="91"/>
+<wire x1="226.06" y1="114.3" x2="226.06" y2="127" width="0.1524" layer="91"/>
+<pinref part="PCB1" gate="G$1" pin="GND@5"/>
+<wire x1="218.44" y1="127" x2="226.06" y2="127" width="0.1524" layer="91"/>
+<wire x1="226.06" y1="127" x2="226.06" y2="137.16" width="0.1524" layer="91"/>
+<pinref part="PCB1" gate="G$1" pin="GPIO18"/>
+<wire x1="218.44" y1="137.16" x2="226.06" y2="137.16" width="0.1524" layer="91"/>
+<wire x1="226.06" y1="137.16" x2="226.06" y2="144.78" width="0.1524" layer="91"/>
+<pinref part="PCB1" gate="G$1" pin="GND@8"/>
+<wire x1="226.06" y1="144.78" x2="218.44" y2="144.78" width="0.1524" layer="91"/>
+<pinref part="PCB1" gate="G$1" pin="GND@7"/>
+<wire x1="218.44" y1="109.22" x2="226.06" y2="109.22" width="0.1524" layer="91"/>
+<junction x="226.06" y="109.22"/>
+<junction x="226.06" y="114.3"/>
+<junction x="226.06" y="127"/>
+<junction x="226.06" y="137.16"/>
+</segment>
+<segment>
+<pinref part="U1" gate="A" pin="GND"/>
+<pinref part="GND2" gate="1" pin="GND"/>
+<wire x1="20.32" y1="88.9" x2="17.78" y2="88.9" width="0.1524" layer="91"/>
+<wire x1="17.78" y1="88.9" x2="17.78" y2="81.28" width="0.1524" layer="91"/>
+</segment>
+</net>
+<net name="+5V" class="0">
+<segment>
+<pinref part="PCB1" gate="G$1" pin="5V0@1"/>
+<wire x1="218.44" y1="149.86" x2="218.44" y2="157.48" width="0.1524" layer="91"/>
+<pinref part="SUPPLY1" gate="+5V" pin="+5V"/>
+</segment>
+<segment>
+<wire x1="22.86" y1="121.92" x2="15.24" y2="121.92" width="0.1524" layer="91"/>
+<pinref part="SUPPLY2" gate="+5V" pin="+5V"/>
+<wire x1="15.24" y1="121.92" x2="15.24" y2="134.62" width="0.1524" layer="91"/>
+</segment>
+</net>
+<net name="+3V3" class="0">
+<segment>
+<pinref part="PCB1" gate="G$1" pin="3V3@1"/>
+<wire x1="165.1" y1="149.86" x2="165.1" y2="160.02" width="0.1524" layer="91"/>
+<pinref part="+3V1" gate="G$1" pin="+3V3"/>
+</segment>
+<segment>
+<pinref part="U1" gate="A" pin="VCCA"/>
+<pinref part="+3V2" gate="G$1" pin="+3V3"/>
+<wire x1="20.32" y1="124.46" x2="20.32" y2="129.54" width="0.1524" layer="91"/>
+<pinref part="U1" gate="A" pin="OE"/>
+<wire x1="20.32" y1="116.84" x2="20.32" y2="124.46" width="0.1524" layer="91"/>
+<junction x="20.32" y="124.46"/>
+</segment>
+</net>
+<net name="N$1" class="0">
+<segment>
+<pinref part="U1" gate="A" pin="B1"/>
+<pinref part="JP1" gate="A" pin="1"/>
+<wire x1="55.88" y1="121.92" x2="68.58" y2="121.92" width="0.1524" layer="91"/>
+</segment>
+</net>
+<net name="N$2" class="0">
+<segment>
+<pinref part="U1" gate="A" pin="B2"/>
+<pinref part="JP1" gate="A" pin="2"/>
+<wire x1="55.88" y1="119.38" x2="68.58" y2="119.38" width="0.1524" layer="91"/>
+</segment>
+</net>
+<net name="N$3" class="0">
+<segment>
+<pinref part="U1" gate="A" pin="B3"/>
+<pinref part="JP1" gate="A" pin="3"/>
+<wire x1="55.88" y1="116.84" x2="68.58" y2="116.84" width="0.1524" layer="91"/>
+</segment>
+</net>
+<net name="N$4" class="0">
+<segment>
+<pinref part="U1" gate="A" pin="B4"/>
+<pinref part="JP1" gate="A" pin="4"/>
+<wire x1="55.88" y1="114.3" x2="68.58" y2="114.3" width="0.1524" layer="91"/>
+</segment>
+</net>
+<net name="N$5" class="0">
+<segment>
+<pinref part="U1" gate="A" pin="B5"/>
+<pinref part="JP1" gate="A" pin="5"/>
+<wire x1="55.88" y1="111.76" x2="68.58" y2="111.76" width="0.1524" layer="91"/>
+</segment>
+</net>
+<net name="N$6" class="0">
+<segment>
+<pinref part="U1" gate="A" pin="B6"/>
+<pinref part="JP1" gate="A" pin="6"/>
+<wire x1="55.88" y1="109.22" x2="68.58" y2="109.22" width="0.1524" layer="91"/>
+</segment>
+</net>
+<net name="N$7" class="0">
+<segment>
+<pinref part="U1" gate="A" pin="B7"/>
+<pinref part="JP1" gate="A" pin="7"/>
+<wire x1="55.88" y1="106.68" x2="68.58" y2="106.68" width="0.1524" layer="91"/>
+</segment>
+</net>
+<net name="N$8" class="0">
+<segment>
+<pinref part="U1" gate="A" pin="B8"/>
+<pinref part="JP1" gate="A" pin="8"/>
+<wire x1="55.88" y1="104.14" x2="68.58" y2="104.14" width="0.1524" layer="91"/>
+</segment>
+</net>
+<net name="UART_TX" class="0">
+<segment>
+<pinref part="PCB1" gate="G$1" pin="TXD0/GPIO14"/>
+<wire x1="218.44" y1="142.24" x2="231.14" y2="142.24" width="0.1524" layer="91"/>
+<label x="228.6" y="142.24" size="1.778" layer="95"/>
+</segment>
+</net>
+<net name="UART_RX" class="0">
+<segment>
+<pinref part="PCB1" gate="G$1" pin="RXD0/GPIO15"/>
+<wire x1="218.44" y1="139.7" x2="231.14" y2="139.7" width="0.1524" layer="91"/>
+<label x="228.6" y="139.7" size="1.778" layer="95"/>
+</segment>
+</net>
+<net name="SPI_CLK" class="0">
+<segment>
+<pinref part="PCB1" gate="G$1" pin="GPIO11/SCLK"/>
+<wire x1="165.1" y1="121.92" x2="152.4" y2="121.92" width="0.1524" layer="91"/>
+<label x="144.78" y="121.92" size="1.778" layer="95"/>
+</segment>
+</net>
+<net name="SPI_MISO" class="0">
+<segment>
+<pinref part="PCB1" gate="G$1" pin="GPIO09/MISO"/>
+<wire x1="165.1" y1="124.46" x2="152.4" y2="124.46" width="0.1524" layer="91"/>
+<label x="144.78" y="124.46" size="1.778" layer="95"/>
+</segment>
+</net>
+<net name="SPI_MOSI" class="0">
+<segment>
+<pinref part="PCB1" gate="G$1" pin="GPIO10/MOSI"/>
+<wire x1="165.1" y1="127" x2="152.4" y2="127" width="0.1524" layer="91"/>
+<label x="144.78" y="127" size="1.778" layer="95"/>
+</segment>
+</net>
+<net name="N$14" class="0">
+<segment>
+<pinref part="PCB1" gate="G$1" pin="GPIO22/GEN3"/>
+<wire x1="165.1" y1="132.08" x2="162.56" y2="132.08" width="0.1524" layer="91"/>
+<wire x1="162.56" y1="132.08" x2="160.02" y2="129.54" width="0.1524" layer="91"/>
+<wire x1="160.02" y1="129.54" x2="152.4" y2="129.54" width="0.1524" layer="91"/>
+</segment>
+</net>
 </nets>
 </sheet>
@@
 </schematic>
 </drawing>
+<compatibility>
+<note version="6.3" minversion="6.2.2" severity="warning">
+Since Version 6.2.2 text objects can contain more than one line,
+which will not be processed correctly with this version.
+</note>
+</compatibility>
 </eagle>

Commit message: routing
Parts:
- added BATTERY, MOTOR1, MOTOR2: (no value), pinhead:PINHD-1X2
- added C1, C10, C2, C3, C4, C6: 100n, rcl:C-EUC0603
- added C11, C7, C8, C9: 10n, rcl:C-EUC0603
- added C5: (no value), rcl:CPOL-EU153CLV-0405
- added IC1: 7805TV, linear:7805TV
- added JP2: (no value), pinhead:PINHD-2X20
- added JP3: (no value), pinhead:PINHD-1X4
- added R11, R12, R3, R4, R5, R6, R8, R9: 1K, rcl:R-EU_R0603
- added SERVO: (no value), pinhead:PINHD-1X3
- added U2, U3: SN74LVC1G04DCKR, RPiAutonomousCar:SN74LVC1G04DCKR
- added U4: MCP3004-I/ST, RPiAutonomousCar:MCP3004-I/ST
Connections:
- removed net SPI_CLK: PCB1.GPIO11/SCLK
- removed net SPI_MISO: PCB1.GPIO09/MISO
- removed net SPI_MOSI: PCB1.GPIO10/MOSI
- removed net UART_RX: PCB1.RXD0/GPIO15
- removed net UART_TX: PCB1.TXD0/GPIO14
- new net +UB: BATTERY.2, C4.1, C5.+, IC1.VI, U$1.VM1, U$1.VM2, U$1.VM3
- new net AN_CH0: JP3.1, R5.2
- new net AN_CH1: JP3.2, R3.2
- new net AN_CH2: JP3.3, R8.2
- new net AN_CH3: JP3.4, R11.2
- new net M1_DIR_INV: U$1.AIN2, U2.Y
- new net M1_OUT1: MOTOR1.1, U$1.A01, U$1.A01_2
- new net M1_OUT2: MOTOR1.2, U$1.A02, U$1.A02_2
- new net M2_DIR_INV: U$1.BIN2, U3.Y
- new net M2_OUT1: MOTOR2.1, U$1.B01, U$1.B01_2
- new net M2_OUT2: MOTOR2.2, U$1.B02, U$1.B02_2
- new net N$10: C2.2, U3.VCC
- new net N$11: C11.1, R5.1, R6.2, U4.CH0
- new net N$13: C7.1, R3.1, R4.2, U4.CH1
- new net N$15: C9.1, R11.1, R12.2, U4.CH3
- new net N$9: C1.2, U2.VCC
- new net RPI10: JP2.10, PCB1.RXD0/GPIO15
- new net RPI11: JP2.11, PCB1.GPIO17/GEN0
- new net RPI12: JP2.12, PCB1.GPIO18
- new net RPI13: JP2.13, PCB1.GPIO27/GEN2
- new net RPI14: U1.A7
- new net RPI15: JP2.15, PCB1.GPIO22/GEN3, U1.A8
- new net RPI16: JP2.16, PCB1.GEN4/GPIO23
- new net RPI17: JP2.17
- new net RPI18: JP2.18, PCB1.GEN5/GPIO24
- new net RPI19: JP2.19, PCB1.GPIO10/MOSI, U1.A1, U4.DIN
- new net RPI21: JP2.21, PCB1.GPIO09/MISO, U1.A2, U4.DOUT
- new net RPI22: JP2.22, PCB1.GEN6/GPIO25
- new net RPI23: JP2.23, PCB1.GPIO11/SCLK, U1.A3, U4.CLK
- new net RPI24: JP2.24, PCB1.!CE0!/GPIO08, U1.A4, U4.*CS/SHDN
- new net RPI26: JP2.26, PCB1.!CE!/GPIO07
- new net RPI27: JP2.27, PCB1.ID_SD
- new net RPI28: JP2.28, PCB1.ID_SC
- new net RPI29: JP2.29, PCB1.GPIO05, U$1.PWMA
- new net RPI3: JP2.3, PCB1.GPIO02/SDA1, U1.A5
- new net RPI31: JP2.31, PCB1.GPIO06, U$1.AIN1, U2.A
- new net RPI32: JP2.32, PCB1.GPIO12
- new net RPI33: JP2.33, PCB1.GPIO13, U$1.STBY
- new net RPI35: JP2.35, PCB1.GPIO19, U$1.BIN1, U3.A
- new net RPI36: JP2.36, PCB1.GPIO16
- new net RPI37: JP2.37, PCB1.GPIO26, U$1.PWMB
- new net RPI38: JP2.38, PCB1.GPIO20
- new net RPI40: JP2.40, PCB1.GPIO21
- new net RPI5: JP2.5, PCB1.GPIO03/SCL1, U1.A6
- new net RPI7: JP2.7, PCB1.GPIO04/GCKL
- new net RPI8: JP2.8, PCB1.TXD0/GPIO14
- new net SERVOPWM: SERVO.1
- net +3V3: now also C1.1, C2.1, C3.1, C6.1, JP2.1, PCB1.3V3@2, SERVO.2, U$1.VCC, U4.VDD, U4.VREF
- net +5V: now also C10.1, IC1.VO, JP2.2, JP2.4, U1.VCCB
- net GND: now also BATTERY.1, C10.2, C11.2, C3.2, C4.2, C5.-, C6.2, C7.2, C8.2, C9.2, IC1.GND, JP2.14, JP2.20, JP2.25, JP2.30, JP2.34, JP2.39, JP2.6, JP2.9, PCB1.GND@4, R12.1, R4.1, R6.1, R9.1, SERVO.3, U$1.GND, U$1.PGND1, U$1.PGND1_2, U$1.PGND2, U$1.PGND2_2, U2.GND, U3.GND, U4.AGND, U4.DGND; no longer PCB1.GPIO18
- net N$14: now also C8.1, R8.1, R9.2, U4.CH2; no longer PCB1.GPIO22/GEN3
Other:
- note added: "I2C"
- note added: "SPI"
- note added: "UART"
- moved on the sheet: JP1, PCB1, U$1, U1

Commit message: routing
Parts:
- added C12, C13: 100n, rcl:C-EUC0603
- added I2C_JP2, I2C_JP3: (no value), pinhead:PINHD-1X2
- added LED1: (no value), led:LEDSML0603
- added R1: 1K, rcl:R-EU_R0603
- added SJ1: (no value), jumper:SJ2W
- added SPI_JP2: (no value), pinhead:PINHD-1X3
- R11: value 1K -> 10K
- R12: value 1K -> 22K
Connections:
- new net N$12: LED1.C, R1.1
- new net N$16: LED1.A
- net +3V3: now also C12.1
- net +5V: now also C13.1
- net +UB: now also SJ1.3
- net AN_CH3: now also SJ1.1, SJ1.2
- net GND: now also C12.2, C13.2, R1.2; no longer PCB1.BL, PCB1.TL, PCB1.TR
- net RPI19: now also SPI_JP2.3
- net RPI21: now also SPI_JP2.2
- net RPI23: now also SPI_JP2.1
- net RPI3: now also I2C_JP2.2, I2C_JP3.2
- net RPI5: now also I2C_JP2.1, I2C_JP3.1
Other:
- moved on the sheet: C3, JP1

Commit message: routing ...
Parts:
- removed BATTERY, I2C_JP2, I2C_JP3, MOTOR1, MOTOR2: (no value), pinhead:PINHD-1X2
- removed C10: 100n, rcl:C-EUC0603
- removed IC1: 7805TV, linear:7805TV
- removed SERVO, SPI_JP2: (no value), pinhead:PINHD-1X3
- added JP10, JP11, JP12: (no value), jumper:JP1E
- added JP13, JP4, JP5, JP9: (no value), jumper:JP2E
- added JP6, JP7, JP8: (no value), jumper:JP4E
- JP1: device pinhead:PINHD-1X8 -> jumper:JP1E
Connections:
- removed net RPI14: U1.A7
- removed net RPI17: JP2.17
- removed net SERVOPWM: SERVO.1
- net +3V3: now also JP2.17, JP6.4, JP9.2; no longer SERVO.2
- net +5V: now also JP5.2; no longer C10.1, IC1.VO
- net +UB: now also JP4.2; no longer BATTERY.2, IC1.VI
- net GND: now also JP4.1, JP4.3, JP5.1, JP5.3, JP6.1, JP9.3; no longer BATTERY.1, C10.2, IC1.GND, SERVO.3
- net M1_OUT1: now also JP10.1; no longer MOTOR1.1
- net M1_OUT2: now also JP10.2; no longer MOTOR1.2
- net M2_OUT1: now also JP11.1; no longer MOTOR2.1
- net M2_OUT2: now also JP11.2; no longer MOTOR2.2
- net N$1: now also JP8.4; no longer JP1.8
- net N$16: now also JP9.1; no longer LED1.A
- net N$2: now also JP8.3; no longer JP1.7
- net N$3: now also JP8.2; no longer JP1.6
- net N$4: now also JP8.1; no longer JP1.5
- net N$5: now also JP7.4; no longer JP1.4
- net N$6: now also JP7.3; no longer JP1.3
- net N$7: now also JP7.2; no longer JP1.2
- net N$8: now also JP7.1; no longer JP1.1
- net RPI10: now also U1.A8
- net RPI15: no longer U1.A8
- net RPI19: now also JP13.3; no longer SPI_JP2.3
- net RPI21: now also JP13.2; no longer SPI_JP2.2
- net RPI23: now also JP13.1; no longer SPI_JP2.1
- net RPI3: now also JP1.2, JP12.2; no longer I2C_JP2.2, I2C_JP3.2
- net RPI40: now also LED1.A
- net RPI5: now also JP1.1, JP12.1; no longer I2C_JP2.1, I2C_JP3.1
- net RPI8: now also U1.A7
Other:
- note added: "Antenna jumper"
- note added: "Board Power"
- note added: "Servo Jumper"
- moved on the sheet: C12, C13, C2
