File: 01_Hardware/RPiAutonomousCar.sch (EAGLE design)
At the start: 42 parts, among them U1 TXB0108PWR, U2 SN74LVC1G04DCKR, U3 SN74LVC1G04DCKR, U4 MCP3004-I/ST

Commit message: routing ...
Parts:
- removed JP3: (no value), pinhead:PINHD-1X4
- JP13: device jumper:JP2E -> jumper:JP4E
Connections:
- removed net N$16: JP9.1
- removed net N$3: JP8.2, U1.B6
- new net N$18: JP1.1, JP12.2, JP8.1, U1.B5
- net AN_CH0: now also JP13.1; no longer JP3.1
- net AN_CH1: now also JP13.2; no longer JP3.2
- net AN_CH2: now also JP13.3; no longer JP3.3
- net AN_CH3: now also JP13.4; no longer JP3.4
- net N$4: now also JP1.2, JP12.1, JP8.2, U1.B6; no longer JP8.1, U1.B5
- net RPI19: no longer JP13.3
- net RPI21: no longer JP13.2
- net RPI23: no longer JP13.1
- net RPI26: now also JP6.3
- net RPI27: now also JP6.2
- net RPI3: no longer JP1.2, JP12.2
- net RPI5: no longer JP1.1, JP12.1
- net RPI7: now also JP9.1
Other:
- moved on the sheet: JP1, JP12
Changed lines of the file:
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@@
 <part name="GND10" library="supply1" deviceset="GND" device=""/>
 <part name="+3V7" library="supply1" deviceset="+3V3" device=""/>
-<part name="JP3" library="pinhead" deviceset="PINHD-1X4" device=""/>
 <part name="+3V8" library="supply1" deviceset="+3V3" device=""/>
 <part name="GND11" library="supply1" deviceset="GND" device=""/>
@@
 <part name="JP1" library="jumper" deviceset="JP1E" device=""/>
 <part name="JP12" library="jumper" deviceset="JP1E" device=""/>
-<part name="JP13" library="jumper" deviceset="JP2E" device=""/>
+<part name="JP13" library="jumper" deviceset="JP4E" device=""/>
 </parts>
 <sheets>
 <sheet>
 <plain>
-<text x="20.32" y="147.32" size="1.778" layer="94" rot="R90">SPI</text>
-<text x="20.32" y="139.7" size="1.778" layer="94" rot="R90">I2C</text>
+<text x="20.32" y="142.24" size="1.778" layer="94" rot="R90">SPI</text>
+<text x="20.32" y="137.16" size="1.778" layer="94" rot="R90">I2C</text>
 <text x="20.32" y="129.54" size="1.778" layer="94" rot="R90">UART</text>
 <text x="5.08" y="7.62" size="1.778" layer="90" rot="R90">Board Power</text>
@@
 <instance part="GND10" gate="1" x="180.34" y="38.1"/>
 <instance part="+3V7" gate="G$1" x="215.9" y="58.42"/>
-<instance part="JP3" gate="A" x="256.54" y="86.36"/>
 <instance part="+3V8" gate="G$1" x="38.1" y="53.34"/>
 <instance part="GND11" gate="1" x="38.1" y="33.02"/>
@@
 <instance part="JP7" gate="G$1" x="83.82" y="157.48" rot="R270"/>
 <instance part="JP8" gate="G$1" x="83.82" y="147.32" rot="R270"/>
-<instance part="JP1" gate="A" x="20.32" y="124.46" rot="R90"/>
-<instance part="JP12" gate="A" x="10.16" y="119.38" rot="R90"/>
-<instance part="JP13" gate="1" x="7.62" y="147.32" rot="R90"/>
+<instance part="JP1" gate="A" x="78.74" y="137.16" rot="R270"/>
+<instance part="JP12" gate="A" x="78.74" y="129.54" rot="R270"/>
+<instance part="JP13" gate="G$1" x="256.54" y="88.9" rot="R270"/>
 </instances>
 <busses>
@@
 </segment>
 <segment>
-<wire x1="53.34" y1="17.78" x2="53.34" y2="12.7" width="0.762" layer="92"/>
-<label x="55.88" y="7.62" size="1.778" layer="95" rot="R90"/>
+<wire x1="58.42" y1="15.24" x2="58.42" y2="12.7" width="0.762" layer="92"/>
+<label x="60.96" y="10.16" size="1.778" layer="95" rot="R90"/>
 </segment>
 </bus>
@@
 <segment>
 <pinref part="U1" gate="A" pin="A5"/>
-<wire x1="22.86" y1="139.7" x2="27.94" y2="139.7" width="0.1524" layer="91"/>
+<wire x1="22.86" y1="139.7" x2="33.02" y2="139.7" width="0.1524" layer="91"/>
 <label x="25.4" y="139.7" size="1.778" layer="95"/>
-<wire x1="27.94" y1="139.7" x2="33.02" y2="139.7" width="0.1524" layer="91"/>
-<wire x1="22.86" y1="127" x2="27.94" y2="127" width="0.1524" layer="91"/>
-<wire x1="27.94" y1="127" x2="27.94" y2="139.7" width="0.1524" layer="91"/>
-<junction x="27.94" y="139.7"/>
-<wire x1="12.7" y1="121.92" x2="27.94" y2="121.92" width="0.1524" layer="91"/>
-<wire x1="27.94" y1="121.92" x2="27.94" y2="127" width="0.1524" layer="91"/>
-<junction x="27.94" y="127"/>
-<pinref part="JP1" gate="A" pin="2"/>
-<pinref part="JP12" gate="A" pin="2"/>
 </segment>
 </net>
@@
 <segment>
 <pinref part="U1" gate="A" pin="A6"/>
-<wire x1="22.86" y1="137.16" x2="30.48" y2="137.16" width="0.1524" layer="91"/>
+<wire x1="22.86" y1="137.16" x2="33.02" y2="137.16" width="0.1524" layer="91"/>
 <label x="25.4" y="137.16" size="1.778" layer="95"/>
-<wire x1="30.48" y1="137.16" x2="33.02" y2="137.16" width="0.1524" layer="91"/>
-<wire x1="22.86" y1="124.46" x2="30.48" y2="124.46" width="0.1524" layer="91"/>
-<wire x1="30.48" y1="124.46" x2="30.48" y2="137.16" width="0.1524" layer="91"/>
-<junction x="30.48" y="137.16"/>
-<wire x1="12.7" y1="119.38" x2="30.48" y2="119.38" width="0.1524" layer="91"/>
-<wire x1="30.48" y1="119.38" x2="30.48" y2="124.46" width="0.1524" layer="91"/>
-<junction x="30.48" y="124.46"/>
-<pinref part="JP1" gate="A" pin="1"/>
-<pinref part="JP12" gate="A" pin="1"/>
 </segment>
 </net>
@@
 <label x="101.6" y="162.56" size="1.778" layer="95"/>
 </segment>
+<segment>
+<pinref part="JP9" gate="1" pin="1"/>
+<wire x1="43.18" y1="43.18" x2="40.64" y2="43.18" width="0.1524" layer="91"/>
+<label x="40.64" y="43.18" size="1.778" layer="95" rot="R90"/>
+</segment>
 </net>
 <net name="RPI11" class="0">
@@
 <pinref part="U1" gate="A" pin="A1"/>
 <label x="25.4" y="149.86" size="1.778" layer="95"/>
-<wire x1="10.16" y1="149.86" x2="33.02" y2="149.86" width="0.1524" layer="91"/>
-<pinref part="JP13" gate="1" pin="3"/>
+<wire x1="22.86" y1="149.86" x2="33.02" y2="149.86" width="0.1524" layer="91"/>
 </segment>
 <segment>
@@
 <pinref part="U1" gate="A" pin="A2"/>
 <label x="25.4" y="147.32" size="1.778" layer="95"/>
-<wire x1="10.16" y1="147.32" x2="33.02" y2="147.32" width="0.1524" layer="91"/>
-<pinref part="JP13" gate="1" pin="2"/>
+<wire x1="22.86" y1="147.32" x2="33.02" y2="147.32" width="0.1524" layer="91"/>
 </segment>
 <segment>
@@
 <segment>
 <pinref part="U1" gate="A" pin="A3"/>
-<wire x1="10.16" y1="144.78" x2="33.02" y2="144.78" width="0.1524" layer="91"/>
+<wire x1="22.86" y1="144.78" x2="33.02" y2="144.78" width="0.1524" layer="91"/>
 <label x="25.4" y="144.78" size="1.778" layer="95"/>
-<pinref part="JP13" gate="1" pin="1"/>
 </segment>
 <segment>
@@
 <label x="101.6" y="137.16" size="1.778" layer="95"/>
 </segment>
+<segment>
+<pinref part="JP6" gate="G$1" pin="2"/>
+<wire x1="58.42" y1="12.7" x2="45.72" y2="12.7" width="0.1524" layer="91"/>
+<label x="48.26" y="12.7" size="1.778" layer="95"/>
+</segment>
 </net>
 <net name="RPI29" class="0">
@@
 <wire x1="147.32" y1="139.7" x2="127" y2="139.7" width="0.1524" layer="91"/>
 <label x="134.62" y="139.7" size="1.778" layer="95"/>
+</segment>
+<segment>
+<pinref part="JP6" gate="G$1" pin="3"/>
+<wire x1="58.42" y1="15.24" x2="45.72" y2="15.24" width="0.1524" layer="91"/>
+<label x="48.26" y="15.24" size="1.778" layer="95"/>
 </segment>
 </net>
@@
 </segment>
 <segment>
-<pinref part="JP3" gate="A" pin="1"/>
 <wire x1="254" y1="91.44" x2="243.84" y2="91.44" width="0.1524" layer="91"/>
 <label x="238.76" y="91.44" size="1.778" layer="95"/>
+<pinref part="JP13" gate="G$1" pin="1"/>
 </segment>
 </net>
@@
 </segment>
 <segment>
-<pinref part="JP3" gate="A" pin="2"/>
 <wire x1="254" y1="88.9" x2="243.84" y2="88.9" width="0.1524" layer="91"/>
 <label x="238.76" y="88.9" size="1.778" layer="95"/>
+<pinref part="JP13" gate="G$1" pin="2"/>
 </segment>
 </net>
@@
 </segment>
 <segment>
-<pinref part="JP3" gate="A" pin="3"/>
 <wire x1="254" y1="86.36" x2="243.84" y2="86.36" width="0.1524" layer="91"/>
 <label x="238.76" y="86.36" size="1.778" layer="95"/>
+<pinref part="JP13" gate="G$1" pin="3"/>
 </segment>
 </net>
@@
 </segment>
 <segment>
-<pinref part="JP3" gate="A" pin="4"/>
 <wire x1="254" y1="83.82" x2="238.76" y2="83.82" width="0.1524" layer="91"/>
 <label x="238.76" y="83.82" size="1.778" layer="95"/>
+<pinref part="JP13" gate="G$1" pin="4"/>
 </segment>
 <segment>
@@
 </segment>
 </net>
-<net name="N$3" class="0">
-<segment>
-<pinref part="U1" gate="A" pin="B6"/>
-<wire x1="68.58" y1="147.32" x2="81.28" y2="147.32" width="0.1524" layer="91"/>
-<pinref part="JP8" gate="G$1" pin="2"/>
-</segment>
-</net>
-<net name="N$4" class="0">
-<segment>
-<pinref part="U1" gate="A" pin="B5"/>
-<wire x1="68.58" y1="149.86" x2="81.28" y2="149.86" width="0.1524" layer="91"/>
-<pinref part="JP8" gate="G$1" pin="1"/>
-</segment>
-</net>
 <net name="N$5" class="0">
 <segment>
@@
 </segment>
 </net>
-<net name="N$16" class="0">
-<segment>
-<pinref part="JP9" gate="1" pin="1"/>
-<wire x1="43.18" y1="43.18" x2="40.64" y2="43.18" width="0.1524" layer="91"/>
-</segment>
-</net>
+<net name="N$18" class="0">
+<segment>
+<pinref part="JP12" gate="A" pin="2"/>
+<wire x1="76.2" y1="127" x2="71.12" y2="127" width="0.1524" layer="91"/>
+<wire x1="71.12" y1="127" x2="71.12" y2="137.16" width="0.1524" layer="91"/>
+<pinref part="JP1" gate="A" pin="1"/>
+<wire x1="71.12" y1="137.16" x2="76.2" y2="137.16" width="0.1524" layer="91"/>
+<pinref part="U1" gate="A" pin="B5"/>
+<wire x1="68.58" y1="149.86" x2="71.12" y2="149.86" width="0.1524" layer="91"/>
+<pinref part="JP8" gate="G$1" pin="1"/>
+<wire x1="71.12" y1="149.86" x2="81.28" y2="149.86" width="0.1524" layer="91"/>
+<wire x1="71.12" y1="137.16" x2="71.12" y2="149.86" width="0.1524" layer="91"/>
+<junction x="71.12" y="149.86"/>
+<junction x="71.12" y="137.16"/>
+</segment>
+</net>
+<net name="N$4" class="0">
+<segment>
+<pinref part="JP12" gate="A" pin="1"/>
+<wire x1="76.2" y1="129.54" x2="73.66" y2="129.54" width="0.1524" layer="91"/>
+<wire x1="73.66" y1="129.54" x2="73.66" y2="134.62" width="0.1524" layer="91"/>
+<pinref part="JP1" gate="A" pin="2"/>
+<wire x1="73.66" y1="134.62" x2="76.2" y2="134.62" width="0.1524" layer="91"/>
+<pinref part="U1" gate="A" pin="B6"/>
+<wire x1="68.58" y1="147.32" x2="73.66" y2="147.32" width="0.1524" layer="91"/>
+<pinref part="JP8" gate="G$1" pin="2"/>
+<wire x1="73.66" y1="147.32" x2="81.28" y2="147.32" width="0.1524" layer="91"/>
+<wire x1="73.66" y1="134.62" x2="73.66" y2="147.32" width="0.1524" layer="91"/>
+<junction x="73.66" y="147.32"/>
+<junction x="73.66" y="134.62"/>
+</segment>
+</net>

Commit message: rounting/Pinout minor changes
Parts:
- removed C1, C2: 100n, rcl:C-EUC0603
- removed U2, U3: SN74LVC1G04DCKR, RPiAutonomousCar:SN74LVC1G04DCKR
Connections:
- removed net M1_DIR_INV: U$1.AIN2, U2.Y
- removed net M2_DIR_INV: U$1.BIN2, U3.Y
- removed net N$10: C2.2, U3.VCC
- removed net N$9: C1.2, U2.VCC
- net +3V3: no longer C1.1, C2.1
- net GND: no longer U2.GND, U3.GND
- net RPI12: now also JP6.2
- net RPI13: now also JP6.3
- net RPI22: now also U4.*CS/SHDN
- net RPI24: no longer U4.*CS/SHDN
- net RPI26: no longer JP6.3
- net RPI27: no longer JP6.2
- net RPI31: no longer U2.A
- net RPI32: now also U$1.AIN2
- net RPI35: no longer U3.A
- net RPI36: now also U$1.BIN2
Other:
- moved on the sheet: JP10, JP11, JP4, JP5, JP6, JP9, LED1, R1

Commit message: ready for review
Parts:
- removed JP4, JP5: (no value), jumper:JP2E
- added JP14, JP3: (no value), jumper:JP1E
Connections:
- net +5V: now also JP14.2; no longer JP5.2
- net +UB: now also JP3.2; no longer JP4.2
- net GND: now also JP14.1, JP3.1; no longer JP4.1, JP4.3, JP5.1, JP5.3
Changed lines of the file:
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@@
 <part name="R1" library="rcl" deviceset="R-EU_" device="R0603" value="1K"/>
 <part name="GND1" library="supply1" deviceset="GND" device=""/>
-<part name="JP4" library="jumper" deviceset="JP2E" device=""/>
-<part name="JP5" library="jumper" deviceset="JP2E" device=""/>
 <part name="JP9" library="jumper" deviceset="JP2E" device=""/>
 <part name="JP10" library="jumper" deviceset="JP1E" device=""/>
@@
 <part name="JP12" library="jumper" deviceset="JP1E" device=""/>
 <part name="JP13" library="jumper" deviceset="JP4E" device=""/>
+<part name="JP3" library="jumper" deviceset="JP1E" device=""/>
+<part name="JP14" library="jumper" deviceset="JP1E" device=""/>
 </parts>
 <sheets>
@@
 <instance part="JP2" gate="A" x="121.92" y="147.32"/>
 <instance part="+3V3" gate="G$1" x="109.22" y="177.8"/>
-<instance part="GND3" gate="1" x="88.9" y="116.84"/>
+<instance part="GND3" gate="1" x="88.9" y="114.3"/>
 <instance part="GND4" gate="1" x="154.94" y="114.3"/>
 <instance part="SUPPLY3" gate="+5V" x="142.24" y="172.72"/>
@@
 <instance part="C4" gate="G$1" x="149.86" y="93.98"/>
 <instance part="C5" gate="G$1" x="142.24" y="93.98"/>
-<instance part="GND8" gate="1" x="53.34" y="20.32"/>
+<instance part="GND8" gate="1" x="55.88" y="22.86"/>
 <instance part="SUPPLY5" gate="G$1" x="55.88" y="43.18"/>
 <instance part="U4" gate="A" x="241.3" y="66.04"/>
@@
 <instance part="+3V8" gate="G$1" x="109.22" y="45.72"/>
 <instance part="GND11" gate="1" x="109.22" y="25.4"/>
-<instance part="SUPPLY6" gate="+5V" x="58.42" y="33.02"/>
+<instance part="SUPPLY6" gate="+5V" x="60.96" y="35.56"/>
 <instance part="C12" gate="G$1" x="15.24" y="165.1"/>
 <instance part="C13" gate="G$1" x="7.62" y="165.1"/>
@@
 <instance part="R1" gate="G$1" x="139.7" y="30.48" rot="R270"/>
 <instance part="GND1" gate="1" x="139.7" y="22.86"/>
-<instance part="JP4" gate="1" x="45.72" y="38.1" rot="R90"/>
-<instance part="JP5" gate="1" x="45.72" y="27.94" rot="R90"/>
 <instance part="JP9" gate="1" x="116.84" y="33.02" rot="R270"/>
 <instance part="JP10" gate="A" x="27.94" y="40.64" rot="R270"/>
@@
 <instance part="JP12" gate="A" x="78.74" y="129.54" rot="R270"/>
 <instance part="JP13" gate="G$1" x="256.54" y="88.9" rot="R270"/>
+<instance part="JP3" gate="A" x="48.26" y="35.56" rot="R90"/>
+<instance part="JP14" gate="A" x="48.26" y="27.94" rot="R90"/>
 </instances>
 <busses>
@@
 <segment>
 <pinref part="GND3" gate="1" pin="GND"/>
-<wire x1="88.9" y1="119.38" x2="88.9" y2="121.92" width="0.1524" layer="91"/>
+<wire x1="88.9" y1="116.84" x2="88.9" y2="121.92" width="0.1524" layer="91"/>
 <pinref part="JP2" gate="A" pin="9"/>
 <wire x1="88.9" y1="121.92" x2="88.9" y2="139.7" width="0.1524" layer="91"/>
@@
 </segment>
 <segment>
-<pinref part="JP4" gate="1" pin="3"/>
-<wire x1="48.26" y1="40.64" x2="53.34" y2="40.64" width="0.1524" layer="91"/>
-<wire x1="53.34" y1="40.64" x2="53.34" y2="35.56" width="0.1524" layer="91"/>
-<pinref part="JP4" gate="1" pin="1"/>
-<wire x1="48.26" y1="35.56" x2="53.34" y2="35.56" width="0.1524" layer="91"/>
-<wire x1="53.34" y1="35.56" x2="53.34" y2="30.48" width="0.1524" layer="91"/>
-<pinref part="JP5" gate="1" pin="3"/>
-<wire x1="48.26" y1="30.48" x2="53.34" y2="30.48" width="0.1524" layer="91"/>
-<wire x1="53.34" y1="30.48" x2="53.34" y2="25.4" width="0.1524" layer="91"/>
-<pinref part="JP5" gate="1" pin="1"/>
-<wire x1="48.26" y1="25.4" x2="53.34" y2="25.4" width="0.1524" layer="91"/>
-<wire x1="53.34" y1="25.4" x2="53.34" y2="22.86" width="0.1524" layer="91"/>
 <pinref part="GND8" gate="1" pin="GND"/>
-<junction x="53.34" y="25.4"/>
-<junction x="53.34" y="30.48"/>
-<junction x="53.34" y="35.56"/>
+<pinref part="JP3" gate="A" pin="1"/>
+<wire x1="50.8" y1="35.56" x2="55.88" y2="35.56" width="0.1524" layer="91"/>
+<wire x1="55.88" y1="35.56" x2="55.88" y2="27.94" width="0.1524" layer="91"/>
+<pinref part="JP14" gate="A" pin="1"/>
+<wire x1="55.88" y1="27.94" x2="55.88" y2="25.4" width="0.1524" layer="91"/>
+<wire x1="50.8" y1="27.94" x2="55.88" y2="27.94" width="0.1524" layer="91"/>
+<junction x="55.88" y="27.94"/>
 </segment>
 <segment>
@@
 </segment>
 <segment>
-<pinref part="JP5" gate="1" pin="2"/>
 <pinref part="SUPPLY6" gate="+5V" pin="+5V"/>
-<wire x1="48.26" y1="27.94" x2="58.42" y2="27.94" width="0.1524" layer="91"/>
-<wire x1="58.42" y1="27.94" x2="58.42" y2="30.48" width="0.1524" layer="91"/>
+<wire x1="60.96" y1="30.48" x2="60.96" y2="33.02" width="0.1524" layer="91"/>
+<pinref part="JP14" gate="A" pin="2"/>
+<wire x1="50.8" y1="30.48" x2="60.96" y2="30.48" width="0.1524" layer="91"/>
 </segment>
 </net>
@@
 </segment>
 <segment>
-<pinref part="JP4" gate="1" pin="2"/>
 <pinref part="SUPPLY5" gate="G$1" pin="+UB"/>
-<wire x1="48.26" y1="38.1" x2="55.88" y2="38.1" width="0.1524" layer="91"/>
+<wire x1="50.8" y1="38.1" x2="55.88" y2="38.1" width="0.1524" layer="91"/>
 <wire x1="55.88" y1="38.1" x2="55.88" y2="40.64" width="0.1524" layer="91"/>
-</segment>
-</net>
+<pinref part="JP3" gate="A" pin="2"/>
+</segment>
+</net>
