File: 01_Hardware/RPiAutonomousCar.sch (EAGLE design)
At the start: 37 parts, among them U1 TXB0108PWR, U4 MCP3004-I/ST

Commit message: routing done. Ready to order
Parts:
- added JP4: (no value), jumper:JP1E
- added JP5: (no value), pinhead:PINHD-1X8
- JP7, JP8: device jumper:JP4E -> jumper:JP1E
- R1: value 1K -> x
Connections:
- net +3V3: now also JP7.2, JP8.2
- net +5V: now also JP4.2
- net GND: now also JP4.1, JP7.1, JP8.1
- net N$1: now also JP5.8; no longer JP8.4
- net N$18: now also JP5.5; no longer JP8.1
- net N$2: now also JP5.7; no longer JP8.3
- net N$4: now also JP5.6; no longer JP8.2
- net N$5: now also JP5.4; no longer JP7.4
- net N$6: now also JP5.3; no longer JP7.3
- net N$7: now also JP5.2; no longer JP7.2
- net N$8: now also JP5.1; no longer JP7.1
Changed lines of the file:
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@@
 <part name="GND15" library="supply1" deviceset="GND" device=""/>
 <part name="LED1" library="led" deviceset="LED" device="SML0603"/>
-<part name="R1" library="rcl" deviceset="R-EU_" device="R0603" value="1K"/>
+<part name="R1" library="rcl" deviceset="R-EU_" device="R0603" value="x"/>
 <part name="GND1" library="supply1" deviceset="GND" device=""/>
 <part name="JP9" library="jumper" deviceset="JP2E" device=""/>
@@
 <part name="+3V10" library="supply1" deviceset="+3V3" device=""/>
 <part name="JP6" library="jumper" deviceset="JP4E" device=""/>
-<part name="JP7" library="jumper" deviceset="JP4E" device=""/>
-<part name="JP8" library="jumper" deviceset="JP4E" device=""/>
 <part name="JP1" library="jumper" deviceset="JP1E" device=""/>
 <part name="JP12" library="jumper" deviceset="JP1E" device=""/>
@@
 <part name="JP3" library="jumper" deviceset="JP1E" device=""/>
 <part name="JP14" library="jumper" deviceset="JP1E" device=""/>
+<part name="JP4" library="jumper" deviceset="JP1E" device=""/>
+<part name="JP5" library="pinhead" deviceset="PINHD-1X8" device=""/>
+<part name="JP7" library="jumper" deviceset="JP1E" device=""/>
+<part name="JP8" library="jumper" deviceset="JP1E" device=""/>
+<part name="+3V5" library="supply1" deviceset="+3V3" device=""/>
 </parts>
 <sheets>
@@
 <instance part="C4" gate="G$1" x="149.86" y="93.98"/>
 <instance part="C5" gate="G$1" x="142.24" y="93.98"/>
-<instance part="GND8" gate="1" x="55.88" y="22.86"/>
+<instance part="GND8" gate="1" x="55.88" y="2.54"/>
 <instance part="SUPPLY5" gate="G$1" x="55.88" y="43.18"/>
 <instance part="U4" gate="A" x="241.3" y="66.04"/>
@@
 <instance part="+3V10" gate="G$1" x="83.82" y="43.18"/>
 <instance part="JP6" gate="G$1" x="78.74" y="30.48" rot="R90"/>
-<instance part="JP7" gate="G$1" x="83.82" y="157.48" rot="R270"/>
-<instance part="JP8" gate="G$1" x="83.82" y="147.32" rot="R270"/>
 <instance part="JP1" gate="A" x="78.74" y="137.16" rot="R270"/>
 <instance part="JP12" gate="A" x="78.74" y="129.54" rot="R270"/>
@@
 <instance part="JP3" gate="A" x="48.26" y="35.56" rot="R90"/>
 <instance part="JP14" gate="A" x="48.26" y="27.94" rot="R90"/>
+<instance part="JP4" gate="A" x="48.26" y="22.86" rot="R90"/>
+<instance part="JP5" gate="A" x="83.82" y="149.86"/>
+<instance part="JP7" gate="A" x="48.26" y="12.7" rot="R90"/>
+<instance part="JP8" gate="A" x="48.26" y="7.62" rot="R90"/>
+<instance part="+3V5" gate="G$1" x="60.96" y="20.32"/>
 </instances>
 <busses>
@@
 <wire x1="55.88" y1="35.56" x2="55.88" y2="27.94" width="0.1524" layer="91"/>
 <pinref part="JP14" gate="A" pin="1"/>
-<wire x1="55.88" y1="27.94" x2="55.88" y2="25.4" width="0.1524" layer="91"/>
+<wire x1="55.88" y1="27.94" x2="55.88" y2="22.86" width="0.1524" layer="91"/>
+<wire x1="55.88" y1="22.86" x2="55.88" y2="7.62" width="0.1524" layer="91"/>
+<wire x1="55.88" y1="7.62" x2="55.88" y2="5.08" width="0.1524" layer="91"/>
 <wire x1="50.8" y1="27.94" x2="55.88" y2="27.94" width="0.1524" layer="91"/>
 <junction x="55.88" y="27.94"/>
+<pinref part="JP4" gate="A" pin="1"/>
+<wire x1="50.8" y1="22.86" x2="55.88" y2="22.86" width="0.1524" layer="91"/>
+<pinref part="JP7" gate="A" pin="1"/>
+<wire x1="50.8" y1="12.7" x2="53.34" y2="12.7" width="0.1524" layer="91"/>
+<wire x1="53.34" y1="12.7" x2="53.34" y2="7.62" width="0.1524" layer="91"/>
+<pinref part="JP8" gate="A" pin="1"/>
+<wire x1="50.8" y1="7.62" x2="53.34" y2="7.62" width="0.1524" layer="91"/>
+<wire x1="53.34" y1="7.62" x2="55.88" y2="7.62" width="0.1524" layer="91"/>
+<junction x="53.34" y="7.62"/>
+<junction x="55.88" y="7.62"/>
+<junction x="55.88" y="22.86"/>
 </segment>
 <segment>
@@
 <pinref part="JP14" gate="A" pin="2"/>
 <wire x1="50.8" y1="30.48" x2="60.96" y2="30.48" width="0.1524" layer="91"/>
+<pinref part="JP4" gate="A" pin="2"/>
+<wire x1="50.8" y1="25.4" x2="60.96" y2="25.4" width="0.1524" layer="91"/>
+<wire x1="60.96" y1="25.4" x2="60.96" y2="30.48" width="0.1524" layer="91"/>
+<junction x="60.96" y="30.48"/>
 </segment>
 </net>
@@
 <pinref part="+3V10" gate="G$1" pin="+3V3"/>
 <pinref part="JP6" gate="G$1" pin="4"/>
+</segment>
+<segment>
+<pinref part="JP7" gate="A" pin="2"/>
+<pinref part="+3V5" gate="G$1" pin="+3V3"/>
+<wire x1="50.8" y1="15.24" x2="60.96" y2="15.24" width="0.1524" layer="91"/>
+<wire x1="60.96" y1="15.24" x2="60.96" y2="17.78" width="0.1524" layer="91"/>
+<pinref part="JP8" gate="A" pin="2"/>
+<wire x1="50.8" y1="10.16" x2="60.96" y2="10.16" width="0.1524" layer="91"/>
+<wire x1="60.96" y1="10.16" x2="60.96" y2="15.24" width="0.1524" layer="91"/>
+<junction x="60.96" y="15.24"/>
 </segment>
 </net>
@@
 </segment>
 <segment>
-<wire x1="254" y1="83.82" x2="238.76" y2="83.82" width="0.1524" layer="91"/>
+<wire x1="254" y1="83.82" x2="243.84" y2="83.82" width="0.1524" layer="91"/>
 <label x="238.76" y="83.82" size="1.778" layer="95"/>
 <pinref part="JP13" gate="G$1" pin="4"/>
@@
 <pinref part="U1" gate="A" pin="B8"/>
 <wire x1="68.58" y1="142.24" x2="81.28" y2="142.24" width="0.1524" layer="91"/>
-<pinref part="JP8" gate="G$1" pin="4"/>
+<pinref part="JP5" gate="A" pin="8"/>
 </segment>
 </net>
@@
 <pinref part="U1" gate="A" pin="B7"/>
 <wire x1="68.58" y1="144.78" x2="81.28" y2="144.78" width="0.1524" layer="91"/>
-<pinref part="JP8" gate="G$1" pin="3"/>
+<pinref part="JP5" gate="A" pin="7"/>
 </segment>
 </net>
@@
 <pinref part="U1" gate="A" pin="B4"/>
 <wire x1="68.58" y1="152.4" x2="81.28" y2="152.4" width="0.1524" layer="91"/>
-<pinref part="JP7" gate="G$1" pin="4"/>
+<pinref part="JP5" gate="A" pin="4"/>
 </segment>
 </net>
@@
 <pinref part="U1" gate="A" pin="B3"/>
 <wire x1="68.58" y1="154.94" x2="81.28" y2="154.94" width="0.1524" layer="91"/>
-<pinref part="JP7" gate="G$1" pin="3"/>
+<pinref part="JP5" gate="A" pin="3"/>
 </segment>
 </net>
@@
 <pinref part="U1" gate="A" pin="B2"/>
 <wire x1="68.58" y1="157.48" x2="81.28" y2="157.48" width="0.1524" layer="91"/>
-<pinref part="JP7" gate="G$1" pin="2"/>
+<pinref part="JP5" gate="A" pin="2"/>
 </segment>
 </net>
@@
 <pinref part="U1" gate="A" pin="B1"/>
 <wire x1="68.58" y1="160.02" x2="81.28" y2="160.02" width="0.1524" layer="91"/>
-<pinref part="JP7" gate="G$1" pin="1"/>
+<pinref part="JP5" gate="A" pin="1"/>
 </segment>
 </net>
@@
 <pinref part="U1" gate="A" pin="B5"/>
 <wire x1="68.58" y1="149.86" x2="71.12" y2="149.86" width="0.1524" layer="91"/>
-<pinref part="JP8" gate="G$1" pin="1"/>
 <wire x1="71.12" y1="149.86" x2="81.28" y2="149.86" width="0.1524" layer="91"/>
 <wire x1="71.12" y1="137.16" x2="71.12" y2="149.86" width="0.1524" layer="91"/>
 <junction x="71.12" y="149.86"/>
 <junction x="71.12" y="137.16"/>
+<pinref part="JP5" gate="A" pin="5"/>
 </segment>
 </net>
@@
 <pinref part="U1" gate="A" pin="B6"/>
 <wire x1="68.58" y1="147.32" x2="73.66" y2="147.32" width="0.1524" layer="91"/>
-<pinref part="JP8" gate="G$1" pin="2"/>
 <wire x1="73.66" y1="147.32" x2="81.28" y2="147.32" width="0.1524" layer="91"/>
 <wire x1="73.66" y1="134.62" x2="73.66" y2="147.32" width="0.1524" layer="91"/>
 <junction x="73.66" y="147.32"/>
 <junction x="73.66" y="134.62"/>
-</segment>
-</net>
+<pinref part="JP5" gate="A" pin="6"/>
+</segment>
+</net>
