File: 01_Hardware/REV_A/RPiAutonomousCar.sch (EAGLE design)
At the start: 39 parts, among them U1 TXB0108PWR, U4 MCP3004-I/ST

Commit message: moinor corrections
Parts:
- R11: value 10K -> 22k
- R12: value 22K -> 10k
Changed lines of the file:
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@@
 <part name="R9" library="rcl" deviceset="R-EU_" device="R0603" value="1K"/>
 <part name="C8" library="rcl" deviceset="C-EU" device="C0603" value="10n"/>
-<part name="R11" library="rcl" deviceset="R-EU_" device="R0603" value="10K"/>
-<part name="R12" library="rcl" deviceset="R-EU_" device="R0603" value="22K"/>
+<part name="R11" library="rcl" deviceset="R-EU_" device="R0603" value="22k"/>
+<part name="R12" library="rcl" deviceset="R-EU_" device="R0603" value="10k"/>
 <part name="C9" library="rcl" deviceset="C-EU" device="C0603" value="10n"/>
 <part name="GND10" library="supply1" deviceset="GND" device=""/>
