File: 01_Hardware/REV_B/RPiAutonomousCar.brd (EAGLE design)
At the start: 67.3 x 34 mm, 39 parts, among them U1 TXB0108PWR, U4 MCP3004-I/ST

Commit message: HW Pwm modifications
Connections:
- net +3V3: now also U$1.19
- net RPI29: no longer U$1.23
- net RPI33: no longer U$1.19
- net RPI37: no longer U$1.15
Routing:
- net RPI29: track 25.9 -> 20.9 mm
- net RPI37: track 17.1 -> 15.1 mm
- net RPI33: track 18.7 -> 17.7 mm
Changed lines of the file:
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@@
 <wire x1="41.402" y1="9.906" x2="41.275" y2="9.906" width="0.4064" layer="1"/>
 <wire x1="41.275" y1="9.906" x2="41.275" y2="11.518" width="0.4064" layer="1"/>
-<wire x1="39.37" y1="17.526" x2="30.226" y2="22.098" width="0" layer="19" extent="1-1"/>
+<contactref element="U$1" pad="19"/>
+<wire x1="52.832" y1="11.4935" x2="52.832" y2="12.1285" width="0" layer="19" extent="1-1"/>
+<wire x1="30.226" y1="22.098" x2="39.37" y2="17.526" width="0" layer="19" extent="1-1"/>
 </signal>
 <signal name="RPI3">
@@
 <contactref element="PCB1" pad="29"/>
 <contactref element="JP2" pad="29"/>
-<contactref element="U$1" pad="23"/>
 <wire x1="45.466" y1="22.098" x2="44.958" y2="22.098" width="0.4064" layer="1"/>
 <wire x1="44.958" y1="22.098" x2="44.196" y2="22.86" width="0.4064" layer="1"/>
@@
 <via x="46.99" y="10.414" extent="1-16" drill="0.5"/>
 <wire x1="45.466" y1="20.32" x2="45.466" y2="22.098" width="0.4064" layer="16"/>
-<wire x1="52.832" y1="9.5885" x2="47.8155" y2="9.5885" width="0.4064" layer="1"/>
 <wire x1="47.8155" y1="9.5885" x2="46.99" y2="10.414" width="0.4064" layer="1"/>
 <wire x1="46.99" y1="18.796" x2="46.99" y2="10.414" width="0.4064" layer="16"/>
@@
 <contactref element="PCB1" pad="33"/>
 <contactref element="JP2" pad="33"/>
-<contactref element="U$1" pad="19"/>
 <wire x1="50.546" y1="22.098" x2="50.8" y2="22.098" width="0.4064" layer="16"/>
 <wire x1="50.8" y1="22.098" x2="51.816" y2="23.114" width="0.4064" layer="16"/>
@@
 <wire x1="51.816" y1="25.654" x2="50.546" y2="26.924" width="0.4064" layer="16"/>
 <wire x1="50.546" y1="26.924" x2="50.546" y2="28.116" width="0.4064" layer="16"/>
-<wire x1="52.832" y1="12.1285" x2="51.8795" y2="12.1285" width="0.4064" layer="1"/>
 <via x="51.308" y="13.462" extent="1-16" drill="0.5"/>
 <wire x1="51.308" y1="13.462" x2="51.308" y2="20.574" width="0.4064" layer="16"/>
@@
 <contactref element="PCB1" pad="37"/>
 <contactref element="JP2" pad="37"/>
-<contactref element="U$1" pad="15"/>
 <wire x1="55.626" y1="22.098" x2="56.134" y2="22.098" width="0.4064" layer="16"/>
 <wire x1="56.134" y1="22.098" x2="56.896" y2="22.86" width="0.4064" layer="16"/>
 <wire x1="56.896" y1="22.86" x2="56.896" y2="26.846" width="0.4064" layer="16"/>
 <wire x1="56.896" y1="26.846" x2="55.626" y2="28.116" width="0.4064" layer="16"/>
-<wire x1="52.832" y1="14.6685" x2="54.8005" y2="14.6685" width="0.4064" layer="1"/>
 <wire x1="55.372" y1="15.24" x2="55.372" y2="21.844" width="0.4064" layer="1"/>
 <wire x1="55.372" y1="21.844" x2="55.626" y2="22.098" width="0.4064" layer="1"/>
