File: 01_Hardware/REV_B/RPiAutonomousCar.sch (EAGLE design)
At the start: 39 parts, among them U1 TXB0108PWR, U4 MCP3004-I/ST

Commit message: HW Pwm modifications
Connections:
- net +3V3: now also U$1.STBY
- net RPI29: no longer U$1.PWMA
- net RPI33: no longer U$1.STBY
- net RPI37: no longer U$1.PWMB
Changed lines of the file:
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@@
 <pinref part="U$1" gate="G$1" pin="VCC"/>
 <wire x1="132.08" y1="93.98" x2="132.08" y2="99.06" width="0.1524" layer="91"/>
-<wire x1="106.68" y1="93.98" x2="132.08" y2="93.98" width="0.1524" layer="91"/>
+<wire x1="106.68" y1="93.98" x2="116.84" y2="93.98" width="0.1524" layer="91"/>
 <pinref part="C3" gate="G$1" pin="1"/>
 <junction x="132.08" y="93.98"/>
+<pinref part="U$1" gate="G$1" pin="STBY"/>
+<wire x1="116.84" y1="93.98" x2="132.08" y2="93.98" width="0.1524" layer="91"/>
+<wire x1="106.68" y1="91.44" x2="116.84" y2="91.44" width="0.1524" layer="91"/>
+<wire x1="116.84" y1="91.44" x2="116.84" y2="93.98" width="0.1524" layer="91"/>
+<junction x="116.84" y="93.98"/>
 </segment>
 <segment>
@@
 <label x="101.6" y="134.62" size="1.778" layer="95"/>
 </segment>
-<segment>
-<pinref part="U$1" gate="G$1" pin="PWMA"/>
-<wire x1="127" y1="101.6" x2="106.68" y2="101.6" width="0.1524" layer="91"/>
-<label x="119.38" y="101.6" size="1.778" layer="95"/>
-</segment>
 </net>
 <net name="RPI31" class="0">
@@
 <label x="101.6" y="129.54" size="1.778" layer="95"/>
 </segment>
-<segment>
-<pinref part="U$1" gate="G$1" pin="STBY"/>
-<wire x1="127" y1="91.44" x2="106.68" y2="91.44" width="0.1524" layer="91"/>
-<label x="119.38" y="91.44" size="1.778" layer="95"/>
-</segment>
 </net>
 <net name="RPI35" class="0">
@@
 <label x="101.6" y="124.46" size="1.778" layer="95"/>
 </segment>
-<segment>
-<pinref part="U$1" gate="G$1" pin="PWMB"/>
-<wire x1="127" y1="81.28" x2="106.68" y2="81.28" width="0.1524" layer="91"/>
-<label x="119.38" y="81.28" size="1.778" layer="95"/>
-</segment>
-</net>
+</net>
