File: 01_Hardware/REV_B/REV_B.sch (KiCad schematic (older format))
At the start: 4 parts, among them J1 Conn_02x20_Odd_Even, J2 RPi_GPIO, U1 MCP3004, U2 TB6612FNG

Commit message: Designing RevB
Parts:
- removed J1: Conn_02x20_Odd_Even, Connector_PinHeader_2.54mm:PinHeader_2x20_P2.54mm_Vertical, symbol Connector_Generic:Conn_02x20_Odd_Even
- removed J2: RPi_GPIO, RPi_Hat:Pin_Header_Straight_2x20, symbol REV_B-rescue:RPi_GPIO-RESCUE-REV_B
- removed U1: MCP3004, Package_SSOP:TSSOP-14_4.4x5mm_P0.65mm, symbol Analog_ADC:MCP3004
- removed U2: TB6612FNG, Package_SSOP:SSOP-24_5.3x8.2mm_P0.65mm, symbol Driver_Motor:TB6612FNG
- added 100n1: C, Capacitor_SMD:C_0603_1608Metric, symbol Device:C
- added C1, C2, C3, C4, C5, C6, C7, C8: 10n, Capacitor_SMD:C_0603_1608Metric, symbol Device:C
- added C10: 100n, Capacitor_SMD:C_0603_1608Metric, symbol Device:C
- added C9: 10u, Capacitor_SMD:CP_Elec_4x4.5, symbol Device:CP1_Small
- added J1: RaspberryPi, Connector_PinSocket_2.54mm:PinSocket_2x20_P2.54mm_Vertical, symbol RpiAutonousCar:RaspberryPi
- added J2, J3: Conn_01x02, Connector_Molex:Molex_KK-254_AE-6410-02A_1x02_P2.54mm_Vertical, symbol Connector_Generic:Conn_01x02
- added J4, J5: Conn_01x08_Male, Connector_PinHeader_2.54mm:PinHeader_1x08_P2.54mm_Vertical, symbol Connector_Generic:Conn_01x08_Male
- added R1, R18, R19, R20, R21, R22, R23, R24, R25, R26, R27, R28, R29, R30, R31, R32, R6, R7, R8, R9: 10k, Resistor_SMD:R_0603_1608Metric, symbol Device:R
- added R10, R11, R12, R13, R2, R3, R4, R5: 1k, Resistor_SMD:R_0603_1608Metric, symbol Device:R
- added R14, R15, R16, R17: 22k, Resistor_SMD:R_0603_1608Metric, symbol Device:R
- added U1: TB6612FNG, Package_SSOP:SSOP-24_5.3x8.2mm_P0.65mm, symbol Driver_Motor:TB6612FNG
- added U2, U3, U4, U5: BSS138PS, Package_TO_SOT_SMD:SOT-363_SC-70-6, symbol RpiAutonousCar:BSS138PS
- added U6: MCP3008, Package_SOIC:SOIC-16_3.9x9.9mm_P1.27mm, symbol Analog_ADC:MCP3008
Connections:
- net labels added: +BATT, I2C1_SCL, IC21_SDA
- net labels removed: GPIO10, GPIO11, GPIO12, GPIO13, GPIO14, GPIO15, GPIO16, GPIO17, GPIO18, GPIO19, GPIO2, GPIO20, GPIO21, GPIO22, GPIO23, GPIO24, GPIO25, GPIO26, GPIO27, GPIO3, GPIO4, GPIO5, GPIO6, GPIO7, GPIO8, GPIO9
- wire segments 100 -> 303

Commit message: Work in Progress
Parts:
- added J10, J11, J12, J13, J14, J15, J6, J7, J8, J9: Conn_01x03, Connector_PinHeader_2.54mm:PinHeader_1x03_P2.54mm_Vertical, symbol Connector_Generic:Conn_01x03
- added J2: Conn_01x02, Connector_Molex:Molex_KK-254_AE-6410-02A_1x02_P2.54mm_Vertical, symbol Connector_Generic:Conn_01x02
- added U3: PCA9685PW, Package_SSOP:TSSOP-28_4.4x9.7mm_P0.65mm, symbol Driver_LED:PCA9685PW
- renumbered C9 to C1, C8 to C10, C10 to C2, C1 to C3, C2 to C4, C3 to C5, C4 to C6, C5 to C7, C6 to C8, C7 to C9, J5 to J16, J2 to J3, J3 to J4, J4 to J5, R2 to R1, R11 to R10, R12 to R11, R13 to R12, R14 to R13, R15 to R14, R16 to R15, R17 to R16, R1 to R17, R3 to R2, R4 to R3, R5 to R4, R6 to R5, R7 to R6, R8 to R7, R9 to R8, R10 to R9, U6 to U2, U3 to U5, U2 to U6, U4 to U7, U5 to U8
Connections:
- net labels added: I2C1_SCL_LV, IC21_SDA_LV
- net labels removed: I2C1_SCL, IC21_SDA
- wire segments 303 -> 355
Other:
- moved on the sheet: U2

Commit message: Brd redo due to kicad update
Parts:
- removed J12: Conn_01x03, Connector_PinHeader_2.54mm:PinHeader_1x03_P2.54mm_Vertical, symbol Connector_Generic:Conn_01x03
- U1: footprint Package_SSOP:SSOP-24_5.3x8.2mm_P0.65mm -> Package_SO:SSOP-24_5.3x8.2mm_P0.65mm
- U2: footprint Package_SOIC:SOIC-16_3.9x9.9mm_P1.27mm -> Package_SO:SOIC-16_3.9x9.9mm_P1.27mm
- U3: footprint Package_SSOP:TSSOP-28_4.4x9.7mm_P0.65mm -> Package_SO:TSSOP-28_4.4x9.7mm_P0.65mm
Connections:
- wire segments 355 -> 349
Changed lines of the file:
@@
 F 0 "U1" H 3150 6928 50  0000 C CNN
 F 1 "TB6612FNG" H 3150 6837 50  0000 C CNN
-F 2 "Package_SSOP:SSOP-24_5.3x8.2mm_P0.65mm" H 3600 6350 50  0001 C CNN
+F 2 "Package_SO:SSOP-24_5.3x8.2mm_P0.65mm" H 3600 6350 50  0001 C CNN
 F 3 "https://toshiba.semicon-storage.com/us/product/linear/motordriver/detail.TB6612FNG.html" H 3600 6350 50  0001 C CNN
 	1    3150 5750
@@
 	1900 4700 2050 4700
 Wire Wire Line
-	2050 4700 2050 6150
+	2050 4700 2050 6050
 Wire Wire Line
 	2050 6150 2550 6150
@@
 F 0 "U2" H 3350 3378 50  0000 C CNN
 F 1 "MCP3008" H 3350 3287 50  0000 C CNN
-F 2 "Package_SOIC:SOIC-16_3.9x9.9mm_P1.27mm" H 3450 2800 50  0001 C CNN
+F 2 "Package_SO:SOIC-16_3.9x9.9mm_P1.27mm" H 3450 2800 50  0001 C CNN
 F 3 "http://ww1.microchip.com/downloads/en/DeviceDoc/21295d.pdf" H 3450 2800 50  0001 C CNN
 	1    3350 2700
@@
 F 0 "U3" H 5700 6778 50  0000 C CNN
 F 1 "PCA9685PW" H 5700 6687 50  0000 C CNN
-F 2 "Package_SSOP:TSSOP-28_4.4x9.7mm_P0.65mm" H 5725 4625 50  0001 L CNN
+F 2 "Package_SO:TSSOP-28_4.4x9.7mm_P0.65mm" H 5725 4625 50  0001 L CNN
 F 3 "http://www.nxp.com/documents/data_sheet/PCA9685.pdf" H 5300 6300 50  0001 C CNN
 	1    5700 5600
@@
 	1    0    0    -1
 $EndComp
-$Comp
-L Connector_Generic:Conn_01x03 J12
-U 1 1 5AE2095A
-P 6850 7250
-F 0 "J12" H 6930 7292 50  0000 L CNN
-F 1 "Conn_01x03" H 6930 7201 50  0000 L CNN
-F 2 "Connector_PinHeader_2.54mm:PinHeader_1x03_P2.54mm_Vertical" H 6850 7250 50  0001 C CNN
-F 3 "~" H 6850 7250 50  0001 C CNN
-	1    6850 7250
-	1    0    0    -1
-$EndComp
-Wire Wire Line
-	6400 6400 6400 7150
-Wire Wire Line
-	6400 7150 6650 7150
 Wire Wire Line
 	6400 6300 6430 6300
@@
 	6500 6900 6650 6900
 Connection ~ 6500 6550
-Wire Wire Line
-	6500 6900 6500 7250
-Wire Wire Line
-	6500 7250 6650 7250
-Connection ~ 6500 6900
 Wire Wire Line
 	5700 4600 5700 4550
@@
 	6550 7000 6650 7000
 Connection ~ 6550 6650
-Wire Wire Line
-	6550 7000 6550 7350
-Wire Wire Line
-	6550 7350 6650 7350
 Connection ~ 6550 7000
-Wire Wire Line
-	6550 7350 6550 7550
-Connection ~ 6550 7350
 $Comp
 L power:GND #PWR016
@@
 	4100 4600 3800 4600
 Connection ~ 3800 4600
+Wire Wire Line
+	6550 7000 6550 7550
 $EndSCHEMATC

Commit message: kicad version  REVB added
Parts:
- removed J6, J7, J8: Conn_01x03, Connector_PinHeader_2.54mm:PinHeader_1x03_P2.54mm_Vertical, symbol Connector_Generic:Conn_01x03
- added J14, J15, J16, J17, J18: Conn_01x01, Connector_Pin:Pin_D0.7mm_L6.5mm_W1.8mm_FlatFork, symbol Connector_Generic:Conn_01x01
- added J6: Conn_02x04_Counter_Clockwise, Connector_PinHeader_2.54mm:PinHeader_2x04_P2.54mm_Vertical, symbol Connector_Generic:Conn_02x04_Counter_Clockwise
- C1: renamed from 100n1; value C -> 100n
- J5: footprint Connector_PinHeader_2.54mm:PinHeader_1x08_P2.54mm_Vertical -> Connector_PinHeader_2.54mm:PinHeader_1x08_P2.54mm_Vertical_SMD_Pin1Left
- renumbered C9 to C10, C10 to C11, C1 to C2, C2 to C3, C3 to C4, C4 to C5, C5 to C6, C6 to C7, C7 to C8, C8 to C9, J13 to J10, J14 to J11, J15 to J12, J16 to J13, J11 to J7, J10 to J8, U5 to U4, U6 to U5, U7 to U6, U8 to U7
Connections:
- net labels added: I2C1_SCL_HV, I2C1_SDA_HV, I2C1_SDA_LV, SPI0_CLK_LV, SPI0_CS1_LV, SPI0_MISO_LV, SPI0_MOSI_LV, UART_RX_LV, UART_TX_LV
- net labels removed: IC21_SDA_LV
- wire segments 349 -> 380
Other:
- moved on the sheet: U2

Commit message: Routing started
Parts:
- removed J13: Conn_01x08_Male, Connector_PinHeader_2.54mm:PinHeader_1x08_P2.54mm_Vertical, symbol Connector_Generic:Conn_01x08_Male
- removed J14, J15, J16, J17, J18: Conn_01x01, Connector_Pin:Pin_D0.7mm_L6.5mm_W1.8mm_FlatFork, symbol Connector_Generic:Conn_01x01
- removed J5: Conn_01x08_Male, Connector_PinHeader_2.54mm:PinHeader_1x08_P2.54mm_Vertical_SMD_Pin1Left, symbol Connector_Generic:Conn_01x08_Male
- added D1: LED_CRGB, LED_SMD:LED_Avago_PLCC4_3.2x2.8mm_CW, symbol Device:LED_CRGB
- added J13: Conn_01x08, Connector_PinHeader_2.54mm:PinHeader_1x08_P2.54mm_Vertical, symbol Connector_Generic:Conn_01x08
- added J5: Conn_01x08, Connector_PinHeader_2.54mm:PinHeader_1x08_P2.54mm_Vertical_SMD_Pin1Left, symbol Connector_Generic:Conn_01x08
- added R18, R19, R20, R21, R22, R23, R24, R25, R26, R27, R28, R29: 220, Resistor_SMD:R_0603_1608Metric, symbol Device:R
- added R9: 10k, Resistor_SMD:R_0603_1608Metric, symbol Device:R
- renumbered J9 to J7, J7 to J9, R9 to R10, R10 to R11, R11 to R12, R12 to R13, R13 to R14, R14 to R15, R15 to R16, R16 to R17, R17 to R30, R18 to R31, R19 to R32, R20 to R33, R21 to R34, R22 to R35, R23 to R36, R24 to R37, R25 to R38, R26 to R39, R27 to R40, R28 to R41, R29 to R42, R30 to R43, R31 to R44, R32 to R45
Connections:
- wire segments 380 -> 388

Commit message: Routing almost done
Parts:
- J6: footprint Connector_PinHeader_2.54mm:PinHeader_2x04_P2.54mm_Vertical -> Connector_PinHeader_2.54mm:PinHeader_2x04_P2.54mm_Vertical_SMD
Changed lines of the file:
@@
 F 0 "J6" H 7200 5317 50  0000 C CNN
 F 1 "Conn_02x04_Counter_Clockwise" H 7200 5226 50  0000 C CNN
-F 2 "Connector_PinHeader_2.54mm:PinHeader_2x04_P2.54mm_Vertical" H 7150 5000 50  0001 C CNN
+F 2 "Connector_PinHeader_2.54mm:PinHeader_2x04_P2.54mm_Vertical_SMD" H 7150 5000 50  0001 C CNN
 F 3 "~" H 7150 5000 50  0001 C CNN
 	1    7150 5000

Commit message: Reorder
Parts:
- added R46, R47: 220, Resistor_SMD:R_0603_1608Metric, symbol Device:R
Connections:
- wire segments 388 -> 390
Changed lines of the file:
@@
 L Device:R R29
 U 1 1 5AD8F505
-P 7250 5700
-F 0 "R29" V 7043 5700 50  0000 C CNN
-F 1 "220" V 7134 5700 50  0000 C CNN
-F 2 "Resistor_SMD:R_0603_1608Metric" V 7180 5700 50  0001 C CNN
-F 3 "" H 7250 5700 50  0001 C CNN
-	1    7250 5700
+P 6750 5700
+F 0 "R29" V 6543 5700 50  0000 C CNN
+F 1 "220" V 6634 5700 50  0000 C CNN
+F 2 "Resistor_SMD:R_0603_1608Metric" V 6680 5700 50  0001 C CNN
+F 3 "" H 6750 5700 50  0001 C CNN
+	1    6750 5700
 	0    1    1    0
 $EndComp
@@
 	4800 5650 4800 6700
 Wire Wire Line
-	6400 5700 7100 5700
+	6400 5700 6600 5700
 Wire Wire Line
 	5700 4350 5700 4550
@@
 	5700 4550 5700 4600
 Wire Wire Line
-	7400 5700 7900 5700
+	6900 5700 7900 5700
 Wire Wire Line
 	7900 5800 7200 5800
@@
 	6400 5800 6500 5800
 Wire Wire Line
-	7550 5900 6500 5900
+	7550 5900 6900 5900
 Wire Wire Line
 	6500 5900 6500 5800
@@
 	6400 5900 6450 5900
 Wire Wire Line
-	6450 5900 6450 5950
-Wire Wire Line
-	6450 5950 7150 5950
-Wire Wire Line
-	7150 5950 7150 6200
+	6450 5900 6450 6000
+Wire Wire Line
+	6450 6000 6600 6000
+Wire Wire Line
+	7150 6000 7150 6200
 Wire Wire Line
 	7150 6200 7400 6200
@@
 $EndComp
 Wire Wire Line
-	6400 6000 6850 6000
-Wire Wire Line
-	6850 6000 6850 7300
-Wire Wire Line
 	6850 7300 6750 7300
 Wire Wire Line
-	6400 6100 6800 6100
-Wire Wire Line
-	6800 6100 6800 7100
-Wire Wire Line
 	6800 7100 6750 7100
-Wire Wire Line
-	6400 6200 6750 6200
-Wire Wire Line
-	6750 6200 6750 6900
 Wire Wire Line
 	6350 6900 6450 6900
@@
 Wire Wire Line
 	5700 7100 5700 7500
+$Comp
+L Device:R R46
+U 1 1 5AE07CE9
+P 6750 5900
+F 0 "R46" V 6543 5900 50  0000 C CNN
+F 1 "220" V 6634 5900 50  0000 C CNN
+F 2 "Resistor_SMD:R_0603_1608Metric" V 6680 5900 50  0001 C CNN
+F 3 "" H 6750 5900 50  0001 C CNN
+	1    6750 5900
+	0    1    1    0
+$EndComp
+Wire Wire Line
+	6600 5900 6500 5900
+$Comp
+L Device:R R47
+U 1 1 5AE07E45
+P 6750 6000
+F 0 "R47" V 6543 6000 50  0000 C CNN
+F 1 "220" V 6634 6000 50  0000 C CNN
+F 2 "Resistor_SMD:R_0603_1608Metric" V 6680 6000 50  0001 C CNN
+F 3 "" H 6750 6000 50  0001 C CNN
+	1    6750 6000
+	0    1    1    0
+$EndComp
+Wire Wire Line
+	6900 6000 7150 6000
+Wire Wire Line
+	6400 6400 6750 6400
+Wire Wire Line
+	6750 6400 6750 6900
+Wire Wire Line
+	6400 6300 6800 6300
+Wire Wire Line
+	6800 6300 6800 7100
+Wire Wire Line
+	6850 6200 6850 7300
+Wire Wire Line
+	6400 6200 6850 6200
 $EndSCHEMATC

Commit message: Taster added. routing not done
Parts:
- added R48: 1k, Resistor_SMD:R_0603_1608Metric, symbol Device:R
- added SW1: SW_Push, Button_Switch_SMD:SW_SPST_EVQP7C, symbol Switch:SW_Push
Connections:
- wire segments 390 -> 394
Changed lines of the file:
@@
 Wire Wire Line
 	6400 6200 6850 6200
+$Comp
+L Switch:SW_Push SW1
+U 1 1 5B12BD88
+P 6900 1300
+F 0 "SW1" H 6900 1585 50  0000 C CNN
+F 1 "SW_Push" H 6900 1494 50  0000 C CNN
+F 2 "Button_Switch_SMD:SW_SPST_EVQP7C" H 6900 1500 50  0001 C CNN
+F 3 "" H 6900 1500 50  0001 C CNN
+	1    6900 1300
+	1    0    0    -1
+$EndComp
+$Comp
+L Device:R R48
+U 1 1 5B12BF04
+P 7350 1300
+F 0 "R48" H 7420 1346 50  0000 L CNN
+F 1 "1k" H 7420 1255 50  0000 L CNN
+F 2 "Resistor_SMD:R_0603_1608Metric" V 7280 1300 50  0001 C CNN
+F 3 "" H 7350 1300 50  0001 C CNN
+	1    7350 1300
+	0    1    1    0
+$EndComp
+Wire Wire Line
+	7100 1300 7200 1300
+$Comp
+L power:+3.3V #PWR0101
+U 1 1 5B17FFC3
+P 6600 1200
+F 0 "#PWR0101" H 6600 1050 50  0001 C CNN
+F 1 "+3.3V" H 6615 1373 50  0000 C CNN
+F 2 "" H 6600 1200 50  0001 C CNN
+F 3 "" H 6600 1200 50  0001 C CNN
+	1    6600 1200
+	1    0    0    -1
+$EndComp
+Wire Wire Line
+	6600 1200 6600 1300
+Wire Wire Line
+	6600 1300 6700 1300
+Wire Wire Line
+	7500 1300 7700 1300
 $EndSCHEMATC
