File: 01_Hardware/REV_B/REV_B.sch (KiCad schematic (older format))
At the start: 81 parts, among them J1 RaspberryPi, J10 Conn_01x03, J11 Conn_01x03, J12 Conn_01x03, J13 Conn_01x08, J2 Conn_01x02, J3 Conn_01x02, J4 Conn_01x02, J5 Conn_01x08, J6 Conn_02x04_Counter_Clockwise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

Commit message: routing in progress
Connections:
- net labels added: PUSH_BUTTON
- wire segments 394 -> 395
Changed lines of the file:
@@
 L Switch:SW_Push SW1
 U 1 1 5B12BD88
-P 6900 1300
-F 0 "SW1" H 6900 1585 50  0000 C CNN
-F 1 "SW_Push" H 6900 1494 50  0000 C CNN
-F 2 "Button_Switch_SMD:SW_SPST_EVQP7C" H 6900 1500 50  0001 C CNN
-F 3 "" H 6900 1500 50  0001 C CNN
-	1    6900 1300
+P 7700 1000
+F 0 "SW1" H 7700 1285 50  0000 C CNN
+F 1 "SW_Push" H 7700 1194 50  0000 C CNN
+F 2 "Button_Switch_SMD:SW_SPST_EVQP7C" H 7700 1200 50  0001 C CNN
+F 3 "" H 7700 1200 50  0001 C CNN
+	1    7700 1000
 	1    0    0    -1
 $EndComp
@@
 L Device:R R48
 U 1 1 5B12BF04
-P 7350 1300
-F 0 "R48" H 7420 1346 50  0000 L CNN
-F 1 "1k" H 7420 1255 50  0000 L CNN
-F 2 "Resistor_SMD:R_0603_1608Metric" V 7280 1300 50  0001 C CNN
-F 3 "" H 7350 1300 50  0001 C CNN
-	1    7350 1300
-	0    1    1    0
+P 7300 1000
+F 0 "R48" H 7370 1046 50  0000 L CNN
+F 1 "1k" H 7370 955 50  0000 L CNN
+F 2 "Resistor_SMD:R_0603_1608Metric" V 7230 1000 50  0001 C CNN
+F 3 "" H 7300 1000 50  0001 C CNN
+	1    7300 1000
+	0    -1   -1   0
 $EndComp
 Wire Wire Line
-	7100 1300 7200 1300
+	7500 1000 7450 1000
 $Comp
 L power:+3.3V #PWR0101
 U 1 1 5B17FFC3
-P 6600 1200
-F 0 "#PWR0101" H 6600 1050 50  0001 C CNN
-F 1 "+3.3V" H 6615 1373 50  0000 C CNN
-F 2 "" H 6600 1200 50  0001 C CNN
-F 3 "" H 6600 1200 50  0001 C CNN
-	1    6600 1200
+P 8050 850
+F 0 "#PWR0101" H 8050 700 50  0001 C CNN
+F 1 "+3.3V" H 8065 1023 50  0000 C CNN
+F 2 "" H 8050 850 50  0001 C CNN
+F 3 "" H 8050 850 50  0001 C CNN
+	1    8050 850
 	1    0    0    -1
 $EndComp
 Wire Wire Line
-	6600 1200 6600 1300
+	8050 850  8050 1000
 Wire Wire Line
-	6600 1300 6700 1300
+	8050 1000 7900 1000
 Wire Wire Line
-	7500 1300 7700 1300
+	7150 1000 6950 1000
+Text GLabel 6950 1000 0    50   Input ~ 0
+PUSH_BUTTON
+Text GLabel 2150 3100 2    50   Input ~ 0
+PUSH_BUTTON
+Wire Wire Line
+	1900 3100 2150 3100
 $EndSCHEMATC

Commit message: Routing done
Parts:
- added C12: 0.33u, Capacitor_SMD:C_0603_1608Metric, symbol Device:C
- added C13: 10n, Capacitor_SMD:C_0603_1608Metric, symbol Device:C
- added U8: L7805, Package_TO_SOT_SMD:TO-252-3_TabPin2, symbol Regulator_Linear:L7805
Connections:
- wire segments 395 -> 407
Changed lines of the file:
@@
 Wire Wire Line
 	1900 3100 2150 3100
+$Comp
+L Regulator_Linear:L7805 U8
+U 1 1 5B12AECD
+P 1200 6150
+F 0 "U8" H 1200 6392 50  0000 C CNN
+F 1 "L7805" H 1200 6301 50  0000 C CNN
+F 2 "Package_TO_SOT_SMD:TO-252-3_TabPin2" H 1225 6000 50  0001 L CIN
+F 3 "http://www.st.com/content/ccc/resource/technical/document/datasheet/41/4f/b3/b0/12/d4/47/88/CD00000444.pdf/files/CD00000444.pdf/jcr:content/translations/en.CD00000444.pdf" H 1200 6100 50  0001 C CNN
+	1    1200 6150
+	1    0    0    -1
+$EndComp
+$Comp
+L Device:C C13
+U 1 1 5B12B512
+P 1550 6400
+F 0 "C13" H 1665 6446 50  0000 L CNN
+F 1 "10n" H 1665 6355 50  0000 L CNN
+F 2 "Capacitor_SMD:C_0603_1608Metric" H 1588 6250 50  0001 C CNN
+F 3 "" H 1550 6400 50  0001 C CNN
+	1    1550 6400
+	1    0    0    -1
+$EndComp
+$Comp
+L Device:C C12
+U 1 1 5B12B69A
+P 800 6400
+F 0 "C12" H 915 6446 50  0000 L CNN
+F 1 "0.33u" H 915 6355 50  0000 L CNN
+F 2 "Capacitor_SMD:C_0603_1608Metric" H 838 6250 50  0001 C CNN
+F 3 "" H 800 6400 50  0001 C CNN
+	1    800  6400
+	1    0    0    -1
+$EndComp
+$Comp
+L power:GND #PWR0102
+U 1 1 5B12B786
+P 1200 6700
+F 0 "#PWR0102" H 1200 6450 50  0001 C CNN
+F 1 "GND" H 1205 6527 50  0000 C CNN
+F 2 "" H 1200 6700 50  0001 C CNN
+F 3 "" H 1200 6700 50  0001 C CNN
+	1    1200 6700
+	1    0    0    -1
+$EndComp
+Wire Wire Line
+	800  6250 800  6150
+Wire Wire Line
+	800  6150 900  6150
+Wire Wire Line
+	1500 6150 1550 6150
+Wire Wire Line
+	1550 6150 1550 6250
+Wire Wire Line
+	800  6550 800  6600
+Wire Wire Line
+	800  6600 1200 6600
+Wire Wire Line
+	1550 6600 1550 6550
+Wire Wire Line
+	1200 6700 1200 6600
+Connection ~ 1200 6600
+Wire Wire Line
+	1200 6600 1550 6600
+Wire Wire Line
+	1200 6450 1200 6600
+$Comp
+L power:+5V #PWR0103
+U 1 1 5B12F9C0
+P 1550 6050
+F 0 "#PWR0103" H 1550 5900 50  0001 C CNN
+F 1 "+5V" H 1565 6223 50  0000 C CNN
+F 2 "" H 1550 6050 50  0001 C CNN
+F 3 "" H 1550 6050 50  0001 C CNN
+	1    1550 6050
+	1    0    0    -1
+$EndComp
+$Comp
+L power:+BATT #PWR0104
+U 1 1 5B12FC6B
+P 800 6050
+F 0 "#PWR0104" H 800 5900 50  0001 C CNN
+F 1 "+BATT" H 815 6223 50  0000 C CNN
+F 2 "" H 800 6050 50  0001 C CNN
+F 3 "" H 800 6050 50  0001 C CNN
+	1    800  6050
+	1    0    0    -1
+$EndComp
+Wire Wire Line
+	800  6050 800  6150
+Connection ~ 800  6150
+Wire Wire Line
+	1550 6050 1550 6150
+Connection ~ 1550 6150
 $EndSCHEMATC

Commit message: Routing done. Ready to be manufactured
Parts:
- removed D1: LED_CRGB, LED_SMD:LED_Avago_PLCC4_3.2x2.8mm_CW, symbol Device:LED_CRGB
- added D1: LED_ARGB, LED_SMD:LED_Avago_PLCC4_3.2x2.8mm_CW, symbol Device:LED_ARGB
- added J14: Conn_01x01, Connector_PinHeader_2.54mm:PinHeader_1x01_P2.54mm_Vertical, symbol Connector_Generic:Conn_01x01
- J5: footprint Connector_PinHeader_2.54mm:PinHeader_1x08_P2.54mm_Vertical_SMD_Pin1Left -> Connector_PinHeader_2.54mm:PinHeader_1x08_P2.54mm_Vertical_SMD_Pin1Right
Connections:
- wire segments 407 -> 420
Changed lines of the file:
@@
 	3350 6850 3450 6850
-Wire Wire Line
-	3450 6850 3450 6750
 Wire Wire Line
 	3150 7000 3150 6850
@@
 Connection ~ 3450 4600
 Wire Wire Line
-	3800 5050 3800 4950
-Wire Wire Line
 	4100 4950 4100 5050
 $Comp
@@
 $EndComp
 Wire Wire Line
-	9300 800  9300 750
-Wire Wire Line
 	9550 1000 9550 750
 Wire Wire Line
-	9550 750  9300 750
-Connection ~ 9300 750
-Wire Wire Line
-	9300 750  9300 700
-Wire Wire Line
 	9550 1100 9300 1100
 Wire Wire Line
@@
 Wire Wire Line
 	9150 1200 9150 750
-Wire Wire Line
-	9150 750  9300 750
 Wire Wire Line
 	9550 1300 9550 1500
@@
 $EndComp
 Wire Wire Line
-	9250 1850 9250 1800
-Wire Wire Line
 	9500 2050 9500 1800
-Wire Wire Line
-	9500 1800 9250 1800
-Connection ~ 9250 1800
-Wire Wire Line
-	9250 1800 9250 1750
 Wire Wire Line
 	9500 2150 9250 2150
@@
 Wire Wire Line
 	9100 2250 9100 1800
-Wire Wire Line
-	9100 1800 9250 1800
 Wire Wire Line
 	9500 2350 9500 2550
@@
 $EndComp
 Wire Wire Line
-	9350 4050 9350 4000
-Wire Wire Line
 	9600 4250 9600 4000
 Wire Wire Line
-	9600 4000 9350 4000
-Connection ~ 9350 4000
-Wire Wire Line
-	9350 4000 9350 3950
-Wire Wire Line
 	9600 4350 9350 4350
 Wire Wire Line
@@
 Wire Wire Line
 	9200 4450 9200 4000
-Wire Wire Line
-	9200 4000 9350 4000
 Wire Wire Line
 	9600 4550 9600 4750
@@
 L power:+3.3V #PWR020
 U 1 1 5A7366D3
-P 9300 2850
-F 0 "#PWR020" H 9300 2700 50  0001 C CNN
-F 1 "+3.3V" H 9315 3023 50  0000 C CNN
-F 2 "" H 9300 2850 50  0001 C CNN
-F 3 "" H 9300 2850 50  0001 C CNN
-	1    9300 2850
+P 9300 2800
+F 0 "#PWR020" H 9300 2650 50  0001 C CNN
+F 1 "+3.3V" H 9315 2973 50  0000 C CNN
+F 2 "" H 9300 2800 50  0001 C CNN
+F 3 "" H 9300 2800 50  0001 C CNN
+	1    9300 2800
 	1    0    0    -1
 $EndComp
@@
 	9550 2900 9300 2900
 Connection ~ 9300 2900
-Wire Wire Line
-	9300 2900 9300 2850
 Wire Wire Line
 	9550 3250 9300 3250
@@
 $EndComp
 Wire Wire Line
-	3500 3550 3500 3450
-Wire Wire Line
 	3200 3300 3200 3450
 Wire Wire Line
 	3200 3450 3500 3450
-Connection ~ 3500 3450
-Wire Wire Line
-	3500 3450 3500 3300
 $Comp
 L power:+3.3V #PWR08
@@
 $EndComp
 Wire Wire Line
-	3750 1550 3750 1650
-Wire Wire Line
 	3200 2200 3200 2000
 Wire Wire Line
@@
 	3500 2000 3500 2200
 Wire Wire Line
-	3750 1650 3350 1650
-Wire Wire Line
 	3350 1650 3350 2000
-Connection ~ 3750 1650
 Wire Wire Line
 	3750 1650 3750 1700
@@
 L power:GND #PWR015
 U 1 1 5A7BB0A2
-P 5700 7500
-F 0 "#PWR015" H 5700 7250 50  0001 C CNN
-F 1 "GND" H 5705 7327 50  0000 C CNN
-F 2 "" H 5700 7500 50  0001 C CNN
-F 3 "" H 5700 7500 50  0001 C CNN
-	1    5700 7500
+P 5700 6800
+F 0 "#PWR015" H 5700 6550 50  0001 C CNN
+F 1 "GND" H 5705 6627 50  0000 C CNN
+F 2 "" H 5700 6800 50  0001 C CNN
+F 3 "" H 5700 6800 50  0001 C CNN
+	1    5700 6800
 	1    0    0    -1
 $EndComp
@@
 Connection ~ 10150 6150
 Wire Wire Line
-	5700 6700 5700 7100
-Wire Wire Line
 	6400 4900 6600 4900
 Wire Wire Line
@@
 $EndComp
 Wire Wire Line
-	3700 4350 3350 4350
+	3700 4350 3565 4350
 Connection ~ 3350 4350
 Wire Wire Line
@@
 Wire Wire Line
 	3600 4950 3800 4950
-Connection ~ 3800 4950
 Wire Wire Line
 	3800 4950 3800 4900
@@
 Wire Wire Line
 	6400 5600 6600 5600
-$Comp
-L Driver_LED:PCA9685PW U3
-U 1 1 5A73ACB0
-P 5700 5600
-F 0 "U3" H 5700 6778 50  0000 C CNN
-F 1 "PCA9685PW" H 5700 6687 50  0000 C CNN
-F 2 "Package_SO:TSSOP-28_4.4x9.7mm_P0.65mm" H 5725 4625 50  0001 L CNN
-F 3 "http://www.nxp.com/documents/data_sheet/PCA9685.pdf" H 5300 6300 50  0001 C CNN
-	1    5700 5600
-	1    0    0    -1
-$EndComp
 Text GLabel 2750 2600 1    50   Input ~ 0
 SPI0_CLK_LV
@@
 F 0 "J5" H 6780 2892 50  0000 L CNN
 F 1 "Conn_01x08" H 6780 2801 50  0000 L CNN
-F 2 "Connector_PinHeader_2.54mm:PinHeader_1x08_P2.54mm_Vertical_SMD_Pin1Left" H 6700 2900 50  0001 C CNN
+F 2 "Connector_PinHeader_2.54mm:PinHeader_1x08_P2.54mm_Vertical_SMD_Pin1Right" H 6700 2900 50  0001 C CNN
 F 3 "~" H 6700 2900 50  0001 C CNN
 	1    6700 2900
@@
 Connection ~ 4800 5650
 Wire Wire Line
-	4800 5650 4800 6700
+	4800 5650 4800 5800
 Wire Wire Line
 	6400 5700 6600 5700
@@
 	7350 6100 7350 6400
 Connection ~ 7350 6400
-$Comp
-L Device:LED_CRGB D1
-U 1 1 5B05ADA8
-P 6150 7100
-F 0 "D1" H 6150 7597 50  0000 C CNN
-F 1 "LED_CRGB" H 6150 7506 50  0000 C CNN
-F 2 "LED_SMD:LED_Avago_PLCC4_3.2x2.8mm_CW" H 6150 7050 50  0001 C CNN
-F 3 "~" H 6150 7050 50  0001 C CNN
-	1    6150 7100
-	1    0    0    -1
-$EndComp
 $Comp
 L Device:R R20
@@
 Wire Wire Line
 	6800 7100 6750 7100
-Wire Wire Line
-	6350 6900 6450 6900
-Wire Wire Line
-	6350 7100 6450 7100
-Wire Wire Line
-	6350 7300 6450 7300
-Wire Wire Line
-	5950 7100 5700 7100
-Connection ~ 5700 7100
-Wire Wire Line
-	5700 7100 5700 7500
 $Comp
 L Device:R R46
@@
 	1550 6050 1550 6150
 Connection ~ 1550 6150
+Wire Wire Line
+	6350 6900 6450 6900
+Wire Wire Line
+	6350 7100 6450 7100
+Wire Wire Line
+	6350 7300 6450 7300
+Wire Wire Line
+	5950 7100 5850 7100
+Wire Wire Line
+	5850 7100 5850 6900
+$Comp
+L power:+5V #PWR0105
+U 1 1 5B280780
+P 5850 6900
+F 0 "#PWR0105" H 5850 6750 50  0001 C CNN
+F 1 "+5V" H 5865 7073 50  0000 C CNN
+F 2 "" H 5850 6900 50  0001 C CNN
+F 3 "" H 5850 6900 50  0001 C CNN
+	1    5850 6900
+	1    0    0    -1
+$EndComp
+$Comp
+L Device:LED_ARGB D1
+U 1 1 5B282168
+P 6150 7100
+F 0 "D1" H 6150 6633 50  0000 C CNN
+F 1 "LED_ARGB" H 6150 6724 50  0000 C CNN
+F 2 "LED_SMD:LED_Avago_PLCC4_3.2x2.8mm_CW" H 6150 7050 50  0001 C CNN
+F 3 "~" H 6150 7050 50  0001 C CNN
+	1    6150 7100
+	-1   0    0    1
+$EndComp
+Wire Wire Line
+	5000 5800 4800 5800
+Connection ~ 4800 5800
+Wire Wire Line
+	4800 5800 4800 5900
+Wire Wire Line
+	5000 5900 4800 5900
+Connection ~ 4800 5900
+Wire Wire Line
+	4800 5900 4800 6100
+Wire Wire Line
+	5000 6100 4800 6100
+Connection ~ 4800 6100
+Wire Wire Line
+	4800 6100 4800 6300
+Wire Wire Line
+	5000 6300 4800 6300
+Connection ~ 4800 6300
+Wire Wire Line
+	4800 6300 4800 6700
+$Comp
+L power:+5V #PWR0106
+U 1 1 5B214226
+P 4950 5700
+F 0 "#PWR0106" H 4950 5550 50  0001 C CNN
+F 1 "+5V" H 4965 5873 50  0000 C CNN
+F 2 "" H 4950 5700 50  0001 C CNN
+F 3 "" H 4950 5700 50  0001 C CNN
+	1    4950 5700
+	1    0    0    -1
+$EndComp
+Wire Wire Line
+	5000 6000 4950 6000
+Wire Wire Line
+	4950 6000 4950 5700
+Wire Wire Line
+	5000 6200 4950 6200
+Wire Wire Line
+	4950 6200 4950 6000
+Connection ~ 4950 6000
+Wire Wire Line
+	3450 6750 3450 6850
+Wire Wire Line
+	9300 2800 9300 2900
+Wire Wire Line
+	9150 750  9300 750
+Wire Wire Line
+	9300 750  9300 800
+Wire Wire Line
+	9300 750  9550 750
+Connection ~ 9300 750
+Wire Wire Line
+	9300 700  9300 750
+Wire Wire Line
+	9100 1800 9250 1800
+Wire Wire Line
+	9250 1800 9250 1850
+Wire Wire Line
+	9250 1800 9500 1800
+Connection ~ 9250 1800
+Wire Wire Line
+	9250 1750 9250 1800
+Wire Wire Line
+	9200 4000 9350 4000
+Wire Wire Line
+	9350 4000 9350 4050
+Wire Wire Line
+	9350 4000 9600 4000
+Connection ~ 9350 4000
+Wire Wire Line
+	9350 4000 9350 3950
+Wire Wire Line
+	3350 1650 3750 1650
+Wire Wire Line
+	3750 1650 3750 1550
+Connection ~ 3750 1650
+Wire Wire Line
+	3800 4950 3800 5050
+Connection ~ 3800 4950
+Wire Wire Line
+	3500 3550 3500 3450
+Wire Wire Line
+	3500 3450 3500 3300
+Connection ~ 3500 3450
+Wire Wire Line
+	5700 6800 5700 6700
+$Comp
+L Driver_LED:PCA9685PW U3
+U 1 1 5A73ACB0
+P 5700 5600
+F 0 "U3" H 5700 6778 50  0000 C CNN
+F 1 "PCA9685PW" H 5700 6687 50  0000 C CNN
+F 2 "Package_SO:TSSOP-28_4.4x9.7mm_P0.65mm" H 5725 4625 50  0001 L CNN
+F 3 "http://www.nxp.com/documents/data_sheet/PCA9685.pdf" H 5300 6300 50  0001 C CNN
+	1    5700 5600
+	1    0    0    -1
+$EndComp
+$Comp
+L Connector_Generic:Conn_01x01 J14
+U 1 1 5B15D87F
+P 3565 4150
+F 0 "J14" V 3531 4062 50  0000 R CNN
+F 1 "Conn_01x01" V 3440 4062 50  0000 R CNN
+F 2 "Connector_PinHeader_2.54mm:PinHeader_1x01_P2.54mm_Vertical" H 3565 4150 50  0001 C CNN
+F 3 "~" H 3565 4150 50  0001 C CNN
+	1    3565 4150
+	0    -1   -1   0
+$EndComp
+Connection ~ 3565 4350
+Wire Wire Line
+	3565 4350 3350 4350
 $EndSCHEMATC

Commit message: Last Modification: Jumper J5 long pad smd used
Parts:
- added JP1: Jumper_3_Open, Jumper:SolderJumper-3_P1.3mm_Open_RoundedPad1.0x1.5mm, symbol Jumper:Jumper_3_Open
- J5: footprint Connector_PinHeader_2.54mm:PinHeader_1x08_P2.54mm_Vertical_SMD_Pin1Right -> FSE:PinHeader_1x08_P2.54mm_LongPad_Vertical_SMD_Pin1Right
Connections:
- wire segments 420 -> 426
Changed lines of the file:
@@
 L power:GND #PWR012
 U 1 1 5A78FF7E
-P 4800 6700
-F 0 "#PWR012" H 4800 6450 50  0001 C CNN
-F 1 "GND" H 4805 6527 50  0000 C CNN
-F 2 "" H 4800 6700 50  0001 C CNN
-F 3 "" H 4800 6700 50  0001 C CNN
-	1    4800 6700
+P 4800 6970
+F 0 "#PWR012" H 4800 6720 50  0001 C CNN
+F 1 "GND" H 4805 6797 50  0000 C CNN
+F 2 "" H 4800 6970 50  0001 C CNN
+F 3 "" H 4800 6970 50  0001 C CNN
+	1    4800 6970
 	1    0    0    -1
 $EndComp
@@
 F 0 "J5" H 6780 2892 50  0000 L CNN
 F 1 "Conn_01x08" H 6780 2801 50  0000 L CNN
-F 2 "Connector_PinHeader_2.54mm:PinHeader_1x08_P2.54mm_Vertical_SMD_Pin1Right" H 6700 2900 50  0001 C CNN
+F 2 "FSE:PinHeader_1x08_P2.54mm_LongPad_Vertical_SMD_Pin1Right" H 6700 2900 50  0001 C CNN
 F 3 "~" H 6700 2900 50  0001 C CNN
 	1    6700 2900
@@
 L Switch:SW_Push SW1
 U 1 1 5B12BD88
-P 7700 1000
-F 0 "SW1" H 7700 1285 50  0000 C CNN
-F 1 "SW_Push" H 7700 1194 50  0000 C CNN
-F 2 "Button_Switch_SMD:SW_SPST_EVQP7C" H 7700 1200 50  0001 C CNN
-F 3 "" H 7700 1200 50  0001 C CNN
-	1    7700 1000
+P 2050 7100
+F 0 "SW1" H 2050 7385 50  0000 C CNN
+F 1 "SW_Push" H 2050 7294 50  0000 C CNN
+F 2 "Button_Switch_SMD:SW_SPST_EVQP7C" H 2050 7300 50  0001 C CNN
+F 3 "" H 2050 7300 50  0001 C CNN
+	1    2050 7100
 	1    0    0    -1
 $EndComp
@@
 L Device:R R48
 U 1 1 5B12BF04
-P 7300 1000
-F 0 "R48" H 7370 1046 50  0000 L CNN
-F 1 "1k" H 7370 955 50  0000 L CNN
-F 2 "Resistor_SMD:R_0603_1608Metric" V 7230 1000 50  0001 C CNN
-F 3 "" H 7300 1000 50  0001 C CNN
-	1    7300 1000
+P 1650 7100
+F 0 "R48" H 1720 7146 50  0000 L CNN
+F 1 "1k" H 1720 7055 50  0000 L CNN
+F 2 "Resistor_SMD:R_0603_1608Metric" V 1580 7100 50  0001 C CNN
+F 3 "" H 1650 7100 50  0001 C CNN
+	1    1650 7100
 	0    -1   -1   0
 $EndComp
 Wire Wire Line
-	7500 1000 7450 1000
+	1850 7100 1800 7100
 $Comp
 L power:+3.3V #PWR0101
 U 1 1 5B17FFC3
-P 8050 850
-F 0 "#PWR0101" H 8050 700 50  0001 C CNN
-F 1 "+3.3V" H 8065 1023 50  0000 C CNN
-F 2 "" H 8050 850 50  0001 C CNN
-F 3 "" H 8050 850 50  0001 C CNN
-	1    8050 850
-	1    0    0    -1
-$EndComp
-Wire Wire Line
-	8050 850  8050 1000
-Wire Wire Line
-	8050 1000 7900 1000
-Wire Wire Line
-	7150 1000 6950 1000
-Text GLabel 6950 1000 0    50   Input ~ 0
+P 2400 6950
+F 0 "#PWR0101" H 2400 6800 50  0001 C CNN
+F 1 "+3.3V" H 2415 7123 50  0000 C CNN
+F 2 "" H 2400 6950 50  0001 C CNN
+F 3 "" H 2400 6950 50  0001 C CNN
+	1    2400 6950
+	1    0    0    -1
+$EndComp
+Wire Wire Line
+	2400 6950 2400 7100
+Wire Wire Line
+	2400 7100 2250 7100
+Wire Wire Line
+	1500 7100 1300 7100
+Text GLabel 1300 7100 0    50   Input ~ 0
 PUSH_BUTTON
 Text GLabel 2150 3100 2    50   Input ~ 0
@@
 L Regulator_Linear:L7805 U8
 U 1 1 5B12AECD
-P 1200 6150
-F 0 "U8" H 1200 6392 50  0000 C CNN
-F 1 "L7805" H 1200 6301 50  0000 C CNN
-F 2 "Package_TO_SOT_SMD:TO-252-3_TabPin2" H 1225 6000 50  0001 L CIN
-F 3 "http://www.st.com/content/ccc/resource/technical/document/datasheet/41/4f/b3/b0/12/d4/47/88/CD00000444.pdf/files/CD00000444.pdf/jcr:content/translations/en.CD00000444.pdf" H 1200 6100 50  0001 C CNN
-	1    1200 6150
+P 9325 5675
+F 0 "U8" H 9325 5917 50  0000 C CNN
+F 1 "L7805" H 9325 5826 50  0000 C CNN
+F 2 "Package_TO_SOT_SMD:TO-252-3_TabPin2" H 9350 5525 50  0001 L CIN
+F 3 "http://www.st.com/content/ccc/resource/technical/document/datasheet/41/4f/b3/b0/12/d4/47/88/CD00000444.pdf/files/CD00000444.pdf/jcr:content/translations/en.CD00000444.pdf" H 9325 5625 50  0001 C CNN
+	1    9325 5675
 	1    0    0    -1
 $EndComp
@@
 L Device:C C13
 U 1 1 5B12B512
-P 1550 6400
-F 0 "C13" H 1665 6446 50  0000 L CNN
-F 1 "10n" H 1665 6355 50  0000 L CNN
-F 2 "Capacitor_SMD:C_0603_1608Metric" H 1588 6250 50  0001 C CNN
-F 3 "" H 1550 6400 50  0001 C CNN
-	1    1550 6400
+P 9675 5925
+F 0 "C13" H 9790 5971 50  0000 L CNN
+F 1 "10n" H 9790 5880 50  0000 L CNN
+F 2 "Capacitor_SMD:C_0603_1608Metric" H 9713 5775 50  0001 C CNN
+F 3 "" H 9675 5925 50  0001 C CNN
+	1    9675 5925
 	1    0    0    -1
 $EndComp
@@
 L Device:C C12
 U 1 1 5B12B69A
-P 800 6400
-F 0 "C12" H 915 6446 50  0000 L CNN
-F 1 "0.33u" H 915 6355 50  0000 L CNN
-F 2 "Capacitor_SMD:C_0603_1608Metric" H 838 6250 50  0001 C CNN
-F 3 "" H 800 6400 50  0001 C CNN
-	1    800  6400
+P 8925 5925
+F 0 "C12" H 9040 5971 50  0000 L CNN
+F 1 "0.33u" H 9040 5880 50  0000 L CNN
+F 2 "Capacitor_SMD:C_0603_1608Metric" H 8963 5775 50  0001 C CNN
+F 3 "" H 8925 5925 50  0001 C CNN
+	1    8925 5925
 	1    0    0    -1
 $EndComp
@@
 L power:GND #PWR0102
 U 1 1 5B12B786
-P 1200 6700
-F 0 "#PWR0102" H 1200 6450 50  0001 C CNN
-F 1 "GND" H 1205 6527 50  0000 C CNN
-F 2 "" H 1200 6700 50  0001 C CNN
-F 3 "" H 1200 6700 50  0001 C CNN
-	1    1200 6700
-	1    0    0    -1
-$EndComp
-Wire Wire Line
-	800  6250 800  6150
-Wire Wire Line
-	800  6150 900  6150
-Wire Wire Line
-	1500 6150 1550 6150
-Wire Wire Line
-	1550 6150 1550 6250
-Wire Wire Line
-	800  6550 800  6600
-Wire Wire Line
-	800  6600 1200 6600
-Wire Wire Line
-	1550 6600 1550 6550
-Wire Wire Line
-	1200 6700 1200 6600
-Connection ~ 1200 6600
-Wire Wire Line
-	1200 6600 1550 6600
-Wire Wire Line
-	1200 6450 1200 6600
+P 9325 6225
+F 0 "#PWR0102" H 9325 5975 50  0001 C CNN
+F 1 "GND" H 9330 6052 50  0000 C CNN
+F 2 "" H 9325 6225 50  0001 C CNN
+F 3 "" H 9325 6225 50  0001 C CNN
+	1    9325 6225
+	1    0    0    -1
+$EndComp
+Wire Wire Line
+	8925 5775 8925 5675
+Wire Wire Line
+	8925 5675 9025 5675
+Wire Wire Line
+	9625 5675 9675 5675
+Wire Wire Line
+	9675 5675 9675 5775
+Wire Wire Line
+	8925 6075 8925 6125
+Wire Wire Line
+	8925 6125 9325 6125
+Wire Wire Line
+	9675 6125 9675 6075
+Wire Wire Line
+	9325 6225 9325 6125
+Connection ~ 9325 6125
+Wire Wire Line
+	9325 6125 9675 6125
+Wire Wire Line
+	9325 5975 9325 6125
 $Comp
 L power:+5V #PWR0103
 U 1 1 5B12F9C0
-P 1550 6050
-F 0 "#PWR0103" H 1550 5900 50  0001 C CNN
-F 1 "+5V" H 1565 6223 50  0000 C CNN
-F 2 "" H 1550 6050 50  0001 C CNN
-F 3 "" H 1550 6050 50  0001 C CNN
-	1    1550 6050
+P 9675 5575
+F 0 "#PWR0103" H 9675 5425 50  0001 C CNN
+F 1 "+5V" H 9690 5748 50  0000 C CNN
+F 2 "" H 9675 5575 50  0001 C CNN
+F 3 "" H 9675 5575 50  0001 C CNN
+	1    9675 5575
 	1    0    0    -1
 $EndComp
@@
 L power:+BATT #PWR0104
 U 1 1 5B12FC6B
-P 800 6050
-F 0 "#PWR0104" H 800 5900 50  0001 C CNN
-F 1 "+BATT" H 815 6223 50  0000 C CNN
-F 2 "" H 800 6050 50  0001 C CNN
-F 3 "" H 800 6050 50  0001 C CNN
-	1    800  6050
-	1    0    0    -1
-$EndComp
-Wire Wire Line
-	800  6050 800  6150
-Connection ~ 800  6150
-Wire Wire Line
-	1550 6050 1550 6150
-Connection ~ 1550 6150
+P 8925 5575
+F 0 "#PWR0104" H 8925 5425 50  0001 C CNN
+F 1 "+BATT" H 8940 5748 50  0000 C CNN
+F 2 "" H 8925 5575 50  0001 C CNN
+F 3 "" H 8925 5575 50  0001 C CNN
+	1    8925 5575
+	1    0    0    -1
+$EndComp
+Wire Wire Line
+	8925 5575 8925 5675
+Connection ~ 8925 5675
+Wire Wire Line
+	9675 5575 9675 5675
+Connection ~ 9675 5675
 Wire Wire Line
 	6350 6900 6450 6900
@@
 	5000 6100 4800 6100
 Connection ~ 4800 6100
-Wire Wire Line
-	4800 6100 4800 6300
-Wire Wire Line
-	5000 6300 4800 6300
-Connection ~ 4800 6300
-Wire Wire Line
-	4800 6300 4800 6700
 $Comp
 L power:+5V #PWR0106
@@
 	5000 6000 4950 6000
 Wire Wire Line
-	4950 6000 4950 5700
+	4950 6000 4950 5725
 Wire Wire Line
 	5000 6200 4950 6200
@@
 Wire Wire Line
 	3565 4350 3350 4350
+Wire Wire Line
+	4800 6100 4800 6800
+Wire Wire Line
+	4750 6425 5000 6425
+Wire Wire Line
+	5000 6425 5000 6300
+Wire Wire Line
+	4600 6675 4600 6800
+Wire Wire Line
+	4600 6800 4800 6800
+Connection ~ 4800 6800
+Wire Wire Line
+	4800 6800 4800 6970
+Wire Wire Line
+	4600 6175 4600 5725
+Wire Wire Line
+	4600 5725 4950 5725
+Connection ~ 4950 5725
+Wire Wire Line
+	4950 5725 4950 5700
+$Comp
+L Jumper:Jumper_3_Open JP1
+U 1 1 5B312307
+P 4600 6425
+F 0 "JP1" V 4646 6511 50  0000 L CNN
+F 1 "Jumper_3_Open" V 4555 6511 50  0000 L CNN
+F 2 "Jumper:SolderJumper-3_P1.3mm_Open_RoundedPad1.0x1.5mm" H 4600 6425 50  0001 C CNN
+F 3 "~" H 4600 6425 50  0001 C CNN
+	1    4600 6425
+	0    -1   -1   0
+$EndComp
 $EndSCHEMATC
