File: 01_Hardware/REV_B/REV_B.sch (KiCad schematic (older format))
At the start: 86 parts, among them J1 RaspberryPi, J10 Conn_01x03, J11 Conn_01x03, J12 Conn_01x03, J13 Conn_01x08, J14 Conn_01x01, J2 Conn_01x02, J3 Conn_01x02, J4 Conn_01x02, J5 Conn_01x08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

Commit message: REVB-02 implemented. (1) Rpi header mirrored (2) New Switch added (THR) (3) New RGB LED
Parts:
- removed D1: LED_ARGB, LED_SMD:LED_Avago_PLCC4_3.2x2.8mm_CW, symbol Device:LED_ARGB
- added U9: ASMT-YTB7-0AA02, LED_SMD:LED_Avago_PLCC6_3x2.8mm, symbol LED:ASMT-YTB7-0AA02
- J14: footprint Connector_PinHeader_2.54mm:PinHeader_1x01_P2.54mm_Vertical -> Connector_PinSocket_2.54mm:PinSocket_1x01_P2.54mm_Vertical
- SW1: footprint Button_Switch_SMD:SW_SPST_EVQP7C -> Button_Switch_THT:SW_PUSH_6mm
Connections:
- wire segments 426 -> 430
Changed lines of the file:
@@
 Connection ~ 3350 4600
-Wire Wire Line
-	3350 4200 3350 4350
 Wire Wire Line
 	3450 4600 3800 4600
@@
 L power:GND #PWR015
 U 1 1 5A7BB0A2
-P 5700 6800
-F 0 "#PWR015" H 5700 6550 50  0001 C CNN
-F 1 "GND" H 5705 6627 50  0000 C CNN
-F 2 "" H 5700 6800 50  0001 C CNN
-F 3 "" H 5700 6800 50  0001 C CNN
-	1    5700 6800
+P 5700 6725
+F 0 "#PWR015" H 5700 6475 50  0001 C CNN
+F 1 "GND" H 5705 6552 50  0000 C CNN
+F 2 "" H 5700 6725 50  0001 C CNN
+F 3 "" H 5700 6725 50  0001 C CNN
+	1    5700 6725
 	1    0    0    -1
 $EndComp
@@
 	1    0    0    -1
 $EndComp
-Wire Wire Line
-	3700 4350 3565 4350
-Connection ~ 3350 4350
-Wire Wire Line
-	3350 4350 3350 4600
-Wire Wire Line
-	3700 4450 3600 4450
-Wire Wire Line
-	3600 4450 3600 4950
 Wire Wire Line
 	3600 4950 3800 4950
@@
 L Device:R R20
 U 1 1 5B05B512
-P 6600 7300
-F 0 "R20" V 6393 7300 50  0000 C CNN
-F 1 "220" V 6484 7300 50  0000 C CNN
-F 2 "Resistor_SMD:R_0603_1608Metric" V 6530 7300 50  0001 C CNN
-F 3 "" H 6600 7300 50  0001 C CNN
-	1    6600 7300
+P 6600 7350
+F 0 "R20" V 6393 7350 50  0000 C CNN
+F 1 "220" V 6484 7350 50  0000 C CNN
+F 2 "Resistor_SMD:R_0603_1608Metric" V 6530 7350 50  0001 C CNN
+F 3 "" H 6600 7350 50  0001 C CNN
+	1    6600 7350
 	0    -1   -1   0
 $EndComp
@@
 L Device:R R19
 U 1 1 5B05B629
-P 6600 7100
-F 0 "R19" V 6393 7100 50  0000 C CNN
-F 1 "220" V 6484 7100 50  0000 C CNN
-F 2 "Resistor_SMD:R_0603_1608Metric" V 6530 7100 50  0001 C CNN
-F 3 "" H 6600 7100 50  0001 C CNN
-	1    6600 7100
+P 6600 7250
+F 0 "R19" V 6393 7250 50  0000 C CNN
+F 1 "220" V 6484 7250 50  0000 C CNN
+F 2 "Resistor_SMD:R_0603_1608Metric" V 6530 7250 50  0001 C CNN
+F 3 "" H 6600 7250 50  0001 C CNN
+	1    6600 7250
 	0    -1   -1   0
 $EndComp
@@
 L Device:R R18
 U 1 1 5B05B6E1
-P 6600 6900
-F 0 "R18" V 6393 6900 50  0000 C CNN
-F 1 "220" V 6484 6900 50  0000 C CNN
-F 2 "Resistor_SMD:R_0603_1608Metric" V 6530 6900 50  0001 C CNN
-F 3 "" H 6600 6900 50  0001 C CNN
-	1    6600 6900
+P 6600 7150
+F 0 "R18" V 6393 7150 50  0000 C CNN
+F 1 "220" V 6484 7150 50  0000 C CNN
+F 2 "Resistor_SMD:R_0603_1608Metric" V 6530 7150 50  0001 C CNN
+F 3 "" H 6600 7150 50  0001 C CNN
+	1    6600 7150
 	0    -1   -1   0
 $EndComp
-Wire Wire Line
-	6850 7300 6750 7300
-Wire Wire Line
-	6800 7100 6750 7100
 $Comp
 L Device:R R46
@@
 	6400 6400 6750 6400
 Wire Wire Line
-	6750 6400 6750 6900
+	6750 6400 6750 7150
 Wire Wire Line
 	6400 6300 6800 6300
 Wire Wire Line
-	6800 6300 6800 7100
-Wire Wire Line
-	6850 6200 6850 7300
-Wire Wire Line
 	6400 6200 6850 6200
-$Comp
-L Switch:SW_Push SW1
-U 1 1 5B12BD88
-P 2050 7100
-F 0 "SW1" H 2050 7385 50  0000 C CNN
-F 1 "SW_Push" H 2050 7294 50  0000 C CNN
-F 2 "Button_Switch_SMD:SW_SPST_EVQP7C" H 2050 7300 50  0001 C CNN
-F 3 "" H 2050 7300 50  0001 C CNN
-	1    2050 7100
-	1    0    0    -1
-$EndComp
 $Comp
 L Device:R R48
@@
 Connection ~ 9675 5675
 Wire Wire Line
-	6350 6900 6450 6900
-Wire Wire Line
-	6350 7100 6450 7100
-Wire Wire Line
-	6350 7300 6450 7300
-Wire Wire Line
-	5950 7100 5850 7100
-Wire Wire Line
-	5850 7100 5850 6900
-$Comp
-L power:+5V #PWR0105
-U 1 1 5B280780
-P 5850 6900
-F 0 "#PWR0105" H 5850 6750 50  0001 C CNN
-F 1 "+5V" H 5865 7073 50  0000 C CNN
-F 2 "" H 5850 6900 50  0001 C CNN
-F 3 "" H 5850 6900 50  0001 C CNN
-	1    5850 6900
-	1    0    0    -1
-$EndComp
-$Comp
-L Device:LED_ARGB D1
-U 1 1 5B282168
-P 6150 7100
-F 0 "D1" H 6150 6633 50  0000 C CNN
-F 1 "LED_ARGB" H 6150 6724 50  0000 C CNN
-F 2 "LED_SMD:LED_Avago_PLCC4_3.2x2.8mm_CW" H 6150 7050 50  0001 C CNN
-F 3 "~" H 6150 7050 50  0001 C CNN
-	1    6150 7100
-	-1   0    0    1
-$EndComp
-Wire Wire Line
 	5000 5800 4800 5800
 Connection ~ 4800 5800
@@
 Connection ~ 3500 3450
 Wire Wire Line
-	5700 6800 5700 6700
+	5700 6725 5700 6700
 $Comp
 L Driver_LED:PCA9685PW U3
@@
 	1    0    0    -1
 $EndComp
-$Comp
-L Connector_Generic:Conn_01x01 J14
-U 1 1 5B15D87F
-P 3565 4150
-F 0 "J14" V 3531 4062 50  0000 R CNN
-F 1 "Conn_01x01" V 3440 4062 50  0000 R CNN
-F 2 "Connector_PinHeader_2.54mm:PinHeader_1x01_P2.54mm_Vertical" H 3565 4150 50  0001 C CNN
-F 3 "~" H 3565 4150 50  0001 C CNN
-	1    3565 4150
-	0    -1   -1   0
-$EndComp
-Connection ~ 3565 4350
-Wire Wire Line
-	3565 4350 3350 4350
 Wire Wire Line
 	4800 6100 4800 6800
@@
 	0    -1   -1   0
 $EndComp
+$Comp
+L LED:ASMT-YTB7-0AA02 U9
+U 1 1 5BBBF6C0
+P 5850 7250
+F 0 "U9" H 5850 6883 50  0000 C CNN
+F 1 "ASMT-YTB7-0AA02" H 5850 6974 50  0000 C CNN
+F 2 "LED_SMD:LED_Avago_PLCC6_3x2.8mm" H 5650 6930 50  0001 L CNN
+F 3 "https://docs.broadcom.com/docs/AV02-3793EN" H 6000 7250 50  0001 L CNN
+	1    5850 7250
+	-1   0    0    1
+$EndComp
+Wire Wire Line
+	6850 6200 6850 7350
+Wire Wire Line
+	6800 6300 6800 7250
+Wire Wire Line
+	6150 7150 6450 7150
+Wire Wire Line
+	6800 7250 6750 7250
+Wire Wire Line
+	6150 7250 6450 7250
+Wire Wire Line
+	6150 7350 6450 7350
+Wire Wire Line
+	6750 7350 6850 7350
+$Comp
+L power:GND #PWR0105
+U 1 1 5BF315B1
+P 5475 7550
+F 0 "#PWR0105" H 5475 7300 50  0001 C CNN
+F 1 "GND" H 5480 7377 50  0000 C CNN
+F 2 "" H 5475 7550 50  0001 C CNN
+F 3 "" H 5475 7550 50  0001 C CNN
+	1    5475 7550
+	1    0    0    -1
+$EndComp
+Wire Wire Line
+	5475 7550 5475 7350
+Wire Wire Line
+	5475 7350 5550 7350
+Wire Wire Line
+	5475 7350 5475 7250
+Wire Wire Line
+	5475 7250 5550 7250
+Connection ~ 5475 7350
+Wire Wire Line
+	5475 7250 5475 7150
+Wire Wire Line
+	5475 7150 5550 7150
+Connection ~ 5475 7250
+$Comp
+L Switch:SW_Push SW1
+U 1 1 5BFC8567
+P 2050 7100
+F 0 "SW1" H 2050 7385 50  0000 C CNN
+F 1 "SW_Push" H 2050 7294 50  0000 C CNN
+F 2 "Button_Switch_THT:SW_PUSH_6mm" H 2050 7300 50  0001 C CNN
+F 3 "" H 2050 7300 50  0001 C CNN
+	1    2050 7100
+	1    0    0    -1
+$EndComp
+Wire Wire Line
+	3350 4200 3350 4450
+Wire Wire Line
+	3700 4350 3600 4350
+Wire Wire Line
+	3600 4350 3600 4950
+Wire Wire Line
+	3700 4450 3475 4450
+Connection ~ 3350 4450
+Wire Wire Line
+	3350 4450 3350 4600
+$Comp
+L Connector_Generic:Conn_01x01 J14
+U 1 1 5BB3B5E1
+P 3475 4250
+F 0 "J14" V 3441 4162 50  0000 R CNN
+F 1 "Conn_01x01" V 3350 4162 50  0000 R CNN
+F 2 "Connector_PinSocket_2.54mm:PinSocket_1x01_P2.54mm_Vertical" H 3475 4250 50  0001 C CNN
+F 3 "~" H 3475 4250 50  0001 C CNN
+	1    3475 4250
+	0    -1   -1   0
+$EndComp
+Connection ~ 3475 4450
+Wire Wire Line
+	3475 4450 3350 4450
 $EndSCHEMATC
