File: 01_Hardware/REV_B/eagle/RPiAutonomousCar.brd (EAGLE design)
At the start: 67.3 x 34 mm, 39 parts, among them U1 TXB0108PWR, U4 MCP3004-I/ST

Commit message: (1) Changes from Lome and Ghana (2) Board Revision B started
Connections:
- net +3V3: no longer U$1.19
- net RPI38: now also U$1.19
Routing:
- net RPI33: track 17.7 -> 7.22 mm, vias 1 -> 0
- net RPI37: track 15.1 -> 7.73 mm
Changed lines of the file:
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@@
 <layer number="17" name="Pads" color="2" fill="1" visible="yes" active="yes"/>
 <layer number="18" name="Vias" color="2" fill="1" visible="yes" active="yes"/>
-<layer number="19" name="Unrouted" color="6" fill="1" visible="no" active="yes"/>
+<layer number="19" name="Unrouted" color="6" fill="1" visible="yes" active="yes"/>
 <layer number="20" name="Dimension" color="15" fill="1" visible="yes" active="yes"/>
 <layer number="21" name="tPlace" color="16" fill="1" visible="yes" active="yes"/>
@@
 <wire x1="41.402" y1="9.906" x2="41.275" y2="9.906" width="0.4064" layer="1"/>
 <wire x1="41.275" y1="9.906" x2="41.275" y2="11.518" width="0.4064" layer="1"/>
-<contactref element="U$1" pad="19"/>
-<wire x1="52.832" y1="11.4935" x2="52.832" y2="12.1285" width="0" layer="19" extent="1-1"/>
-<wire x1="30.226" y1="22.098" x2="39.37" y2="17.526" width="0" layer="19" extent="1-1"/>
+<wire x1="39.37" y1="17.526" x2="30.226" y2="22.098" width="0" layer="19" extent="1-1"/>
 </signal>
 <signal name="RPI3">
@@
 <wire x1="51.816" y1="25.654" x2="50.546" y2="26.924" width="0.4064" layer="16"/>
 <wire x1="50.546" y1="26.924" x2="50.546" y2="28.116" width="0.4064" layer="16"/>
-<via x="51.308" y="13.462" extent="1-16" drill="0.5"/>
-<wire x1="51.308" y1="13.462" x2="51.308" y2="20.574" width="0.4064" layer="16"/>
-<wire x1="51.308" y1="20.574" x2="50.546" y2="21.336" width="0.4064" layer="16"/>
-<wire x1="50.546" y1="21.336" x2="50.546" y2="22.098" width="0.4064" layer="16"/>
-<wire x1="51.8795" y1="12.1285" x2="51.308" y2="12.7" width="0.4064" layer="1"/>
-<wire x1="51.308" y1="12.7" x2="51.308" y2="13.462" width="0.4064" layer="1"/>
+<wire x1="51.308" y1="13.462" x2="51.308" y2="13.462" width="0" layer="19" extent="1-16"/>
+<wire x1="51.308" y1="13.462" x2="51.308" y2="20.574" width="0" layer="19" extent="1-16"/>
+<wire x1="51.308" y1="20.574" x2="50.546" y2="21.336" width="0" layer="19" extent="1-16"/>
+<wire x1="50.546" y1="21.336" x2="50.546" y2="22.098" width="0" layer="19" extent="1-16"/>
+<wire x1="51.8795" y1="12.1285" x2="51.308" y2="12.7" width="0" layer="19" extent="1-16"/>
+<wire x1="51.308" y1="12.7" x2="51.308" y2="13.462" width="0" layer="19" extent="1-16"/>
 </signal>
 <signal name="RPI35">
@@
 <wire x1="56.896" y1="22.86" x2="56.896" y2="26.846" width="0.4064" layer="16"/>
 <wire x1="56.896" y1="26.846" x2="55.626" y2="28.116" width="0.4064" layer="16"/>
-<wire x1="55.372" y1="15.24" x2="55.372" y2="21.844" width="0.4064" layer="1"/>
+<wire x1="55.372" y1="15.24" x2="55.372" y2="21.844" width="0" layer="19" extent="1-16"/>
 <wire x1="55.372" y1="21.844" x2="55.626" y2="22.098" width="0.4064" layer="1"/>
-<wire x1="54.8005" y1="14.6685" x2="55.372" y2="15.24" width="0.4064" layer="1"/>
+<wire x1="54.8005" y1="14.6685" x2="55.372" y2="15.24" width="0" layer="19" extent="1-16"/>
 </signal>
 <signal name="RPI8">
@@
 <wire x1="54.356" y1="27.686" x2="54.356" y2="29.386" width="0.4064" layer="16"/>
 <wire x1="54.356" y1="29.386" x2="55.626" y2="30.656" width="0.4064" layer="16"/>
+<contactref element="U$1" pad="19"/>
+<wire x1="52.832" y1="12.1285" x2="55.626" y2="24.638" width="0" layer="19" extent="1-1"/>
 </signal>
 <signal name="RPI40">
